File: clvHd.brd (EAGLE design)
At the start: 25 x 25 mm, 38 parts, among them U1 ADS1293CISQ/NOPB, X1 BM02B-SRSS-TB, X2 BM07B-SRSS-TB, X3 BM07B-SRSS-TB

Commit message: placement
Parts:
- removed C7, C8: 4.70nF, rcl:C0201
- removed Q1: (no value), crystal:CTS406
- removed R8: 4.99k, rcl:R0201
- added S1: TAC_SWITCHSMD, SparkFun-Retired:TACTILE-SWITCH-SMD
- added U$1: ASE, crystalCustom:ASE
- R7: value 4.99k -> 51
- moved C20 123.5 mm to (15.0, 13.5), turned to 90 degrees
- moved C19 116.7 mm to (16.0, 11.0), turned to 270 degrees
- moved C16 105.0 mm to (16.0, 13.5), turned to 90 degrees
- moved C11 82.8 mm to (7.80, 13.4), turned to 90 degrees
- moved C13 82.4 mm to (17.0, 13.5), turned to 90 degrees
- moved LED2 81.1 mm to (6.00, 6.00), turned to 270 degrees
- moved C12 72.6 mm to (7.20, 12.5), turned to 90 degrees
- moved R15 64.4 mm to (7.20, 13.4), turned to 270 degrees
- moved R14 61.1 mm to (7.40, 14.5), turned to 180 degrees
- moved R13 60.5 mm to (18.0, 11.0), turned to 90 degrees
- moved R11 53.4 mm to (17.0, 11.9), turned to 270 degrees
- moved C10 52.0 mm to (18.0, 13.5), turned to 270 degrees
- moved R12 47.8 mm to (9.00, 7.00)
- moved C9 46.9 mm to (16.0, 12.5), turned to 270 degrees
- moved R10 31.6 mm to (12.0, 8.00), turned to 270 degrees
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Connections:
- removed net EL4N: R7.1
- removed net EL4P: R8.1
- removed net IN4N: C7.2, R7.2
- removed net IN4P: C8.2, R8.2
- removed net N$10: R11.1, U1.21
- removed net RLDIN: U1.11
- removed net V+: X2.1, X3.1
- removed net VSSIO: U1.14
- new net CLK: U1.21, X2.7, X3.7
- new net GND: R7.2, S1.3, S1.4, U$1.1, U$1.2, U1.14
- new net N$5: LED1.A, R7.1
- net GNDA: no longer C7.1, C8.1
- net GNDIO: no longer R11.2
- net N$1: now also R11.1, S1.1, S1.2, U1.25; no longer LED1.A
- net N$4: now also U$1.3; no longer Q1.1
- net N$8: now also U$1.4; no longer Q1.3
- net RLDREF: now also U1.11
- net SYNCB: now also X2.6, X3.6
- net VCCIO: now also LED1.C, R11.2
- net VDD: now also X2.1, X3.1

Commit message: gnd-vdd common
Connections:
- removed net GNDA: C1.1, C12.2, C13.2, C16.2, C2.1, C20.2, C3.1, C4.1, C5.1, C6.1, U1.27
- removed net GNDIO: C19.2, U1.29, X2.2, X3.2
- removed net VCCIO: C19.1, LED1.C, R11.2, R12.2, R13.2, U1.22
- net GND: now also C1.1, C12.2, C13.2, C16.2, C19.2, C2.1, C20.2, C3.1, C4.1, C5.1, C6.1, U1.27, U1.29, X2.2, X3.2
- net VDD: now also C19.1, LED1.C, R11.2, R12.2, R13.2, U1.22
Changed lines of the file:
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@@
 <wire x1="10.6" y1="3.61" x2="10.6" y2="10.3" width="0" layer="19" extent="1-1"/>
-</signal>
-<signal name="GNDIO">
-<contactref element="X3" pad="2"/>
-<contactref element="X2" pad="2"/>
-<contactref element="U1" pad="29"/>
-<contactref element="C19" pad="2"/>
-<wire x1="16" y1="10.75" x2="21.39" y2="14.5" width="0" layer="19" extent="1-1"/>
-<wire x1="11.6" y1="12.7" x2="16" y2="10.75" width="0" layer="19" extent="1-1"/>
-<wire x1="3.61" y1="10.5" x2="11.6" y2="12.7" width="0" layer="19" extent="1-1"/>
 </signal>
 <signal name="DOUT">
@@
 <contactref element="R6" pad="1"/>
 </signal>
-<signal name="GNDA">
-<contactref element="C1" pad="1"/>
-<contactref element="C2" pad="1"/>
-<contactref element="C3" pad="1"/>
-<contactref element="C4" pad="1"/>
-<contactref element="C5" pad="1"/>
-<contactref element="C6" pad="1"/>
-<contactref element="C13" pad="2"/>
-<contactref element="C12" pad="2"/>
-<contactref element="U1" pad="27"/>
-<contactref element="C16" pad="2"/>
-<contactref element="C20" pad="2"/>
-<wire x1="12.8" y1="18.75" x2="13.6" y2="18.75" width="0" layer="19" extent="1-1"/>
-<wire x1="11.9" y1="18.75" x2="12.8" y2="18.75" width="0" layer="19" extent="1-1"/>
-<wire x1="11.1" y1="18.75" x2="11.9" y2="18.75" width="0" layer="19" extent="1-1"/>
-<wire x1="10.2" y1="18.75" x2="11.1" y2="18.75" width="0" layer="19" extent="1-1"/>
-<wire x1="9.3" y1="18.75" x2="10.2" y2="18.75" width="0" layer="19" extent="1-1"/>
-<wire x1="14" y1="13.7" x2="13.6" y2="18.75" width="0" layer="19" extent="1-1"/>
-<wire x1="15" y1="13.75" x2="14" y2="13.7" width="0" layer="19" extent="1-1"/>
-<wire x1="16" y1="13.75" x2="15" y2="13.75" width="0" layer="19" extent="1-1"/>
-<wire x1="17" y1="13.75" x2="16" y2="13.75" width="0" layer="19" extent="1-1"/>
-<wire x1="7.2" y1="12.75" x2="9.3" y2="18.75" width="0" layer="19" extent="1-1"/>
-</signal>
 <signal name="VDD">
+<contactref element="X3" pad="1"/>
+<contactref element="X2" pad="1"/>
+<contactref element="LED1" pad="C"/>
+<contactref element="R12" pad="2"/>
+<contactref element="R13" pad="2"/>
+<contactref element="U1" pad="22"/>
+<contactref element="C19" pad="1"/>
 <contactref element="C9" pad="1"/>
 <contactref element="C10" pad="1"/>
 <contactref element="C13" pad="1"/>
+<contactref element="R11" pad="2"/>
 <contactref element="U1" pad="28"/>
 <contactref element="C16" pad="1"/>
-<contactref element="X3" pad="1"/>
-<contactref element="X2" pad="1"/>
 <wire x1="18" y1="13.75" x2="21.39" y2="15.5" width="0" layer="19" extent="1-1"/>
 <wire x1="17" y1="13.25" x2="18" y2="13.75" width="0" layer="19" extent="1-1"/>
 <wire x1="16" y1="13.25" x2="17" y2="13.25" width="0" layer="19" extent="1-1"/>
 <wire x1="16" y1="12.75" x2="16" y2="13.25" width="0" layer="19" extent="1-1"/>
+<wire x1="16" y1="11.25" x2="16" y2="12.75" width="0" layer="19" extent="1-1"/>
+<wire x1="17" y1="11.645" x2="16" y2="11.25" width="0" layer="19" extent="1-1"/>
+<wire x1="18" y1="11.255" x2="17" y2="11.645" width="0" layer="19" extent="1-1"/>
+<wire x1="14" y1="11.2" x2="16" y2="11.25" width="0" layer="19" extent="1-1"/>
 <wire x1="14" y1="14.2" x2="16" y2="13.25" width="0" layer="19" extent="1-1"/>
-<wire x1="3.61" y1="9.5" x2="14" y2="14.2" width="0" layer="19" extent="1-1"/>
+<wire x1="9.255" y1="7" x2="14" y2="11.2" width="0" layer="19" extent="1-1"/>
+<wire x1="5.25" y1="4" x2="9.255" y2="7" width="0" layer="19" extent="1-1"/>
+<wire x1="3.61" y1="9.5" x2="5.25" y2="4" width="0" layer="19" extent="1-1"/>
 </signal>
 <signal name="IN1P1">
@@
 <wire x1="6.75" y1="6" x2="8.745" y2="7" width="0" layer="19" extent="1-1"/>
 </signal>
-<signal name="VCCIO">
-<contactref element="R12" pad="2"/>
-<contactref element="R13" pad="2"/>
-<contactref element="U1" pad="22"/>
-<contactref element="C19" pad="1"/>
-<contactref element="R11" pad="2"/>
-<contactref element="LED1" pad="C"/>
-<wire x1="17" y1="11.645" x2="18" y2="11.255" width="0" layer="19" extent="1-1"/>
-<wire x1="16" y1="11.25" x2="17" y2="11.645" width="0" layer="19" extent="1-1"/>
-<wire x1="14" y1="11.2" x2="16" y2="11.25" width="0" layer="19" extent="1-1"/>
-<wire x1="9.255" y1="7" x2="14" y2="11.2" width="0" layer="19" extent="1-1"/>
-<wire x1="5.25" y1="4" x2="9.255" y2="7" width="0" layer="19" extent="1-1"/>
-</signal>
 <signal name="N$9">
 <contactref element="U1" pad="26"/>
@@
 </signal>
 <signal name="GND">
+<contactref element="C19" pad="2"/>
+<contactref element="C3" pad="1"/>
+<contactref element="C4" pad="1"/>
+<contactref element="C1" pad="1"/>
+<contactref element="C2" pad="1"/>
+<contactref element="C5" pad="1"/>
+<contactref element="C6" pad="1"/>
+<contactref element="R7" pad="2"/>
+<contactref element="C13" pad="2"/>
+<contactref element="C20" pad="2"/>
+<contactref element="U1" pad="27"/>
+<contactref element="C16" pad="2"/>
+<contactref element="U1" pad="29"/>
+<contactref element="C12" pad="2"/>
 <contactref element="U1" pad="14"/>
+<contactref element="U$1" pad="2"/>
+<contactref element="U$1" pad="1"/>
 <contactref element="S1" pad="3"/>
 <contactref element="S1" pad="4"/>
-<contactref element="U$1" pad="2"/>
-<contactref element="U$1" pad="1"/>
-<contactref element="R7" pad="2"/>
-<wire x1="17.32" y1="6.455" x2="19.42" y2="6.455" width="0" layer="19" extent="1-1"/>
+<contactref element="X3" pad="2"/>
+<contactref element="X2" pad="2"/>
+<wire x1="17" y1="13.75" x2="21.39" y2="14.5" width="0" layer="19" extent="1-1"/>
+<wire x1="16" y1="13.75" x2="17" y2="13.75" width="0" layer="19" extent="1-1"/>
+<wire x1="15" y1="13.75" x2="16" y2="13.75" width="0" layer="19" extent="1-1"/>
+<wire x1="14" y1="13.7" x2="15" y2="13.75" width="0" layer="19" extent="1-1"/>
+<wire x1="11.6" y1="12.7" x2="14" y2="13.7" width="0" layer="19" extent="1-1"/>
+<wire x1="9.2" y1="11.2" x2="11.6" y2="12.7" width="0" layer="19" extent="1-1"/>
+<wire x1="7.2" y1="12.75" x2="9.2" y2="11.2" width="0" layer="19" extent="1-1"/>
+<wire x1="16" y1="10.75" x2="16" y2="13.75" width="0" layer="19" extent="1-1"/>
+<wire x1="3.61" y1="10.5" x2="7.2" y2="12.75" width="0" layer="19" extent="1-1"/>
+<wire x1="17.32" y1="6.455" x2="16" y2="10.75" width="0" layer="19" extent="1-1"/>
+<wire x1="19.42" y1="6.455" x2="17.32" y2="6.455" width="0" layer="19" extent="1-1"/>
+<wire x1="13.6" y1="18.75" x2="14" y2="13.7" width="0" layer="19" extent="1-1"/>
+<wire x1="12.8" y1="18.75" x2="13.6" y2="18.75" width="0" layer="19" extent="1-1"/>
+<wire x1="11.9" y1="18.75" x2="12.8" y2="18.75" width="0" layer="19" extent="1-1"/>
+<wire x1="11.1" y1="18.75" x2="11.9" y2="18.75" width="0" layer="19" extent="1-1"/>
+<wire x1="10.2" y1="18.75" x2="11.1" y2="18.75" width="0" layer="19" extent="1-1"/>
+<wire x1="9.3" y1="18.75" x2="10.2" y2="18.75" width="0" layer="19" extent="1-1"/>
+<wire x1="10.255" y1="6.2" x2="9.2" y2="11.2" width="0" layer="19" extent="1-1"/>
 <wire x1="19.894" y1="1.015" x2="19.42" y2="6.455" width="0" layer="19" extent="1-1"/>
 <wire x1="14.306" y1="1.015" x2="19.894" y2="1.015" width="0" layer="19" extent="1-1"/>
-<wire x1="10.255" y1="6.2" x2="14.306" y2="1.015" width="0" layer="19" extent="1-1"/>
-<wire x1="9.2" y1="11.2" x2="10.255" y2="6.2" width="0" layer="19" extent="1-1"/>
 </signal>
 <signal name="N$1">

Commit message: update
Parts:
- removed C1, C2, C3, C4, C5, C6: 4.70nF, rcl:C0201
- removed R1, R2, R3, R4, R5, R6: 4.99k, rcl:R0201
- removed R9: 51, rcl:R0201
- added TP1, TP10, TP11, TP12, TP13, TP14, TP15, TP16, TP17, TP18, TP19, TP2, TP20, TP3, TP4, TP5, TP6, TP7, TP8, TP9: TEST-POINT3, SparkFun-Connectors:PAD.03X.03
- added TP21: PTR1PAD1-17, testpad:P1-17
- C10, C12: device rcl:C0201 -> rcl:C0402
- R13: device rcl:R0201 -> rclCustom:R0402
- moved LED1 13.0 mm to (18.8, 1.80), turned to 0 degrees
- moved X2 12.6 mm to (12.5, 3.61), turned to 0 degrees
- moved X3 12.6 mm to (12.5, 21.4), turned to 180 degrees
- moved U$1 8.15 mm to (22.0, 14.6), turned to 90 degrees
- moved R12 8.08 mm to (2.50, 11.8), turned to 90 degrees
- moved R7 7.52 mm to (17.3, 4.40)
- moved S1 6.66 mm to (19.6, 9.10), turned to 90 degrees
- moved X1 6.62 mm to (4.41, 7.00), turned to 270 degrees
- moved R13 5.46 mm to (13.5, 7.90), turned to 0 degrees
- moved LED2 5.10 mm to (3.26, 10.3), turned to 90 degrees
- moved R14 1.70 mm to (6.10, 13.4), turned to 270 degrees
- moved C10 1.21 mm to (19.1, 14.0)
- moved R11 1.21 mm to (16.5, 13.0), turned to 90 degrees
- moved C12 1.10 mm to (6.40, 11.8), turned to 270 degrees
- moved C19 1.00 mm to (15.0, 10.9)
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Connections:
- removed net EL1N: R1.1
- removed net EL1P: R2.1
- removed net EL2N: R3.1
- removed net EL2P: R4.1
- removed net EL3N: R5.1
- removed net EL3P: R6.1
- removed net IN1N: C1.2, R1.2, U1.1
- removed net IN1P: C2.2, R2.2, U1.2
- removed net IN2N: C3.2, R3.2, U1.3
- removed net IN2P: C4.2, R4.2, U1.4
- removed net IN3N: C5.2, R5.2, U1.5
- removed net IN3P: C6.2, R6.2, U1.6
- removed net N$5: LED1.A, R7.1
- new net IN1: TP18.1, U1.1
- new net IN2.: TP17.1, U1.2
- new net IN3: TP16.1, U1.3
- new net IN4: TP15.1, U1.4
- new net IN5: TP14.1, U1.5
- new net IN6: TP13.1, U1.6
- net ALARMB: now also TP2.1
- net CLK: now also TP9.1, X2.3, X3.3; no longer X2.7, X3.7
- net CMOUT: now also TP12.1
- net CS: now also TP10.1
- net DIN: now also TP7.1
- net DOUT: now also TP6.1
- net DRDYB: now also TP1.1, U1.20; no longer R9.2
- net GND: now also LED1.A, TP4.1; no longer C1.1, C2.1, C3.1, C4.1, C5.1, C6.1, R7.2
- net N$2: now also LED1.C, R7.2; no longer R9.1, U1.20
- net RLDOUT: now also TP19.1
- net RLDREF: now also TP20.1
- net SCLK: now also TP5.1, X2.6, X3.6; no longer X2.3, X3.3
- net SYNCB: now also TP8.1, X2.7, X3.7; no longer X2.6, X3.6
- net VDD: now also R7.1, TP3.1; no longer LED1.C
- net WCT: now also TP11.1
Routing:
- net VDD: track 0.00 -> 91.5 mm, vias 0 -> 4
- net GND: track 0.00 -> 63.6 mm
- net SCLK: track 0.00 -> 42.3 mm
- net SYNCB: track 0.00 -> 38.8 mm
- net DIN: track 0.00 -> 34.0 mm, vias 0 -> 2
- net CLK: track 0.00 -> 33.1 mm, vias 0 -> 2
- net DOUT: track 0.00 -> 29.0 mm, vias 0 -> 2
- net N$8: track 0.00 -> 11.8 mm, vias 0 -> 2
- net N$4: track 0.00 -> 11.6 mm
- net CS: track 0.00 -> 10.8 mm
- net IN1: track 0.00 -> 10.7 mm, vias 0 -> 1
- net IN6: track 0.00 -> 9.07 mm, vias 0 -> 1
- net IN3: track 0.00 -> 8.98 mm, vias 0 -> 1
- net IN4: track 0.00 -> 7.79 mm, vias 0 -> 1
- net ALARMB: track 0.00 -> 7.66 mm
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- added copper zone on layer 16, net IN1
- added copper zone on layer 16, net IN2.
- added copper zone on layer 16, net IN3
- added copper zone on layer 16, net IN4
- added copper zone on layer 16, net IN5
- added copper zone on layer 16, net IN6
- removed copper zone on layer 16, net IN1P
- removed copper zone on layer 16, net IN1P1
- removed copper zone on layer 16, net IN1P2
- removed copper zone on layer 16, net IN1P3
Other:
- outline, holes or cut-outs redrawn
