File: EMG/clvHd_EMG.sch (EAGLE design)
At the start: 25 parts, among them J1 XF2J-1824-12, J2 XF2J-1824-12, U1 ADS1293CISQ/NOPB

Commit message: almost fully routed
Parts:
- removed AND_IC2: SN74AUP1G08QDCKRQ1, SamacSys_Parts:SN74AUP1G08QDCKRQ1
- added NAND_IC: SN74LVC1G132DCKT, SamacSys_Parts:SN74LVC1G132DCKT
- AND_IC: value SN74ALVC08 -> SN74ALVC08LARGE; device SamacSys_Parts:SN74ALVC08 -> SamacSys_Parts:SN74ALVC08LARGE
Connections:
- removed net GPIO2: J1-17.MS, J2-2.MS
- net A0: now also AND_IC-4.A, J1-16.MS, XOR_IC-3.B; no longer AND_IC-1.A, J1-11.MS, XOR_IC-1.B
- net A1: now also AND_IC-3.A, J1-14.MS, XOR_IC-4.B; no longer AND_IC-2.A, J1-13.MS, XOR_IC-2.B
- net A2: now also AND_IC-2.A, J1-13.MS, XOR_IC-1.B; no longer AND_IC-3.A, J1-14.MS, XOR_IC-3.B
- net A3: now also J1-11.MS, NAND_ICG$1.A, XOR_IC-2.B; no longer AND_IC-4.A, J1-16.MS, XOR_IC-4.B
- net CS: now also AND_IC-1.A, NAND_ICG$1.Y; no longer AND_IC-4.Y, AND_IC2-1.A
- net GND: now also NAND_ICG$2.GND; no longer AND_IC2-PWR.GND
- net GPIO1: now also AND_IC-1.B, J1-17.MS, J2-2.MS; no longer AND_IC2-1.B
- net IN5: now also J1-18.MS, J2-1.MSV
- net IN6: no longer J1-18.MS, J2-1.MSV
- net N$11: now also AND_IC-3.B, AND_IC-4.Y, XOR_IC-4.A; no longer AND_IC-1.Y, AND_IC-2.B, XOR_IC-2.A
- net N$13: now also AND_IC-2.B, AND_IC-3.Y, XOR_IC-1.A; no longer AND_IC-2.Y, AND_IC-3.B, XOR_IC-3.A
- net N$16: now also AND_IC-2.Y, NAND_ICG$1.B, XOR_IC-2.A; no longer AND_IC-3.Y, AND_IC-4.B, XOR_IC-4.A
- net N$5: now also AND_IC-1.Y; no longer AND_IC2-1.Y
- net S0: now also J2-3.MS, XOR_IC-3.Y; no longer J2-8.MS, XOR_IC-1.Y
- net S1: now also J2-5.MS, XOR_IC-4.Y; no longer J2-6.MS, XOR_IC-2.Y
- net S2: now also J2-6.MS, XOR_IC-1.Y; no longer J2-5.MS, XOR_IC-3.Y
- net S3: now also J2-8.MS, XOR_IC-2.Y; no longer J2-3.MS, XOR_IC-4.Y
- net VDD: now also AND_IC-4.B, NAND_ICG$2.VCC, XOR_IC-3.A; no longer AND_IC-1.B, AND_IC2-PWR.VCC, XOR_IC-1.A
Other:
- moved on the sheet: AND_IC-1, AND_IC-2, AND_IC-3, AND_IC-4, XOR_IC-1, XOR_IC-2, XOR_IC-3, XOR_IC-4
