File: EMG/clvHd_EMG.brd (EAGLE design)
At the start: 25 x 20 mm, 23 parts, among them J1 XF2J-1024-12, J2 XF2J-1024-12, U1 ADS1293CISQ/NOPB, X1 BM02B-SRSS-TB

Commit message: update
Parts:
- X1: value BM02B-SRSS-TB -> BM03B-SRSS-TB; device con-JST SH:BM02B-SRSS-TB -> con-JST SH:BM03B-SRSS-TB
- moved L1 6.91 mm to (16.0, 15.2), turned to 0 degrees
- moved L3 5.33 mm to (5.50, 13.1), turned to 180 degrees
- moved X1 4.39 mm to (8.00, 7.00)
- moved C12 3.65 mm to (5.55, 10.6)
- moved R12 3.17 mm to (3.40, 5.35)
- moved J2 2.50 mm to (10.5, 16.3)
- moved C10 2.36 mm to (17.4, 2.25)
- moved C13 2.19 mm to (19.2, 4.50)
- moved R14 2.07 mm to (6.50, 12.2)
- moved J1 2.00 mm to (10.5, 2.20)
- moved U$1 2.00 mm to (17.3, 4.70)
- moved C9 1.68 mm to (17.6, 7.25)
- moved R7 1.65 mm to (18.7, 12.0), turned to 90 degrees
- moved R15 1.61 mm to (7.60, 11.7)
- moved R1 1.59 mm to (3.90, 6.95), turned to 270 degrees
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Connections:
- net IN2. renamed IN2
- net IN6: now also X1.3
Routing:
- net IN6: track 9.93 -> 16.6 mm, vias 1 -> 0
- net N$7: track 1.16 -> 7.80 mm
- net CS: track 9.82 -> 4.83 mm
- net N$6: track 1.30 -> 5.79 mm
- net SYNCB: track 22.5 -> 18.5 mm
- net IN5: track 6.28 -> 10.2 mm
- net IN1: track 7.92 -> 4.39 mm
- net N$2: track 1.25 -> 4.43 mm
- net IN3: track 5.47 -> 2.40 mm
- net IN2: track 4.58 -> 1.86 mm
- net N$5: track 1.98 -> 4.33 mm
- net DIN: track 21.1 -> 23.3 mm
- net RLDREF: track 2.77 -> 4.71 mm
- net GND: track 33.6 -> 35.3 mm, vias 8 -> 9
- net ALARMB: track 3.77 -> 2.11 mm
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- removed copper zone on layer 16, net IN6
Other:
- board size 25 x 20 mm -> 21 x 18.5 mm
- board text added: "ClvHd EMG"
- board text added: "ads1293-4l-fpc-v12"
- board text removed: "2"
- board text removed: "3"
- board text removed: "4"
- board text removed: "6"
- board text removed: "ClvHd"
- board text removed: "ads1293-4l-fpc-v10"

Commit message: update
Parts:
- removed X1: BM03B-SRSS-TB, con-JST SH:BM03B-SRSS-TB
- added AND_IC: SN74ALVC08, SamacSys_Parts:SN74ALVC08
- added AND_IC2: SN74AUP1G08QDCKRQ1, SamacSys_Parts:SOT65P210X110-5N
- added XOR_IC: SN74LVC86A, SamacSys_Parts:SN74LVC86ARGYR
- J1, J2: value XF2J-1024-12 -> XF2J-1824-12; device con-omron:XF2J-1024-12 -> con-omron:XF2J-1824-12
- moved R12 2.02 mm to (5.30, 4.65)
- moved U$1 1.20 mm to (17.3, 5.90)
- moved L2 1.12 mm to (10.5, 5.71)
- moved C9 0.90 mm to (17.6, 8.15)
- moved C10 0.78 mm to (17.9, 2.80), turned to 90 degrees
- moved R10 0.60 mm to (12.8, 5.45), turned to 270 degrees
- moved R13 0.57 mm to (14.4, 6.35), turned to 0 degrees
- moved L3 0.40 mm to (5.10, 13.1)
- moved C20 0.36 mm to (18.4, 9.55)
- moved C13 0.30 mm to (19.2, 4.80)
- moved C16 0.20 mm to (16.4, 11.6)
- moved C19 0.20 mm to (17.6, 11.6)
- turned J1 to 270 degrees
- turned J2 to 90 degrees
Connections:
- new net A0: AND_IC.1, J1.11, XOR_IC.2
- new net A1: AND_IC.4, J1.13, XOR_IC.5
- new net A2: AND_IC.8, J1.14, XOR_IC.9
- new net A3: AND_IC.11, J1.16, XOR_IC.12
- new net GPIO1: AND_IC2.2
- new net GPIO2: J1.17, J2.2
- new net N$11: AND_IC.3, AND_IC.5, XOR_IC.4
- new net N$13: AND_IC.6, AND_IC.9, XOR_IC.8
- new net N$16: AND_IC.10, AND_IC.12, XOR_IC.11
- new net S0: J2.8, XOR_IC.3
- new net S1: J2.6, XOR_IC.6
- new net S2: J2.5, XOR_IC.10
- new net S3: J2.3, XOR_IC.13
- net CLK: now also J1.3, J2.16; no longer J1.8, J2.3
- net CS: now also AND_IC.13, AND_IC2.1; no longer X1.1
- net DIN: now also J1.6, J2.13; no longer J1.5, J2.6
- net DOUT: now also J1.4, J2.15; no longer J1.7, J2.4
- net GND: now also AND_IC.7, AND_IC2.3, J1.12, J1.15, J1.2, J1.5, J1.8, J2.11, J2.14, J2.17, J2.4, J2.7, XOR_IC.7; no longer J1.3, J1.6, J1.9, J2.2, J2.5, J2.8
- net IN6: now also J1.18, J2.1; no longer X1.3
- net N$5: now also AND_IC2.4; no longer X1.2
- net RST: now also J1.10, J2.9; no longer J1.1, J2.10
- net SCLK: now also J1.7, J2.12; no longer J1.4, J2.7
- net SYNCB: now also J1.9, J2.10; no longer J1.2, J2.9
- net VDD: now also AND_IC.14, AND_IC.2, AND_IC2.5, J1.1, J2.18, XOR_IC.1, XOR_IC.14; no longer J1.10, J2.1
Routing:
- net SCLK: track 22.2 -> 4.39 mm, vias 2 -> 0
- net GPIO2: track 0.00 -> 16.6 mm, vias 0 -> 2
- net IN6: track 16.6 -> 33.1 mm, vias 0 -> 2
- net GND: track 35.3 -> 28.2 mm, vias 9 -> 3
- net VDD: track 52.6 -> 46.6 mm
- net N$5: track 4.33 -> 0.00 mm
- net RST: track 35.5 -> 31.4 mm
- net CS: track 4.83 -> 1.48 mm
- net CLK: track 22.5 -> 21.3 mm
- net N$8: track 4.93 -> 3.85 mm
- net N$6: track 5.79 -> 4.83 mm
- net N$4: track 7.64 -> 6.97 mm
- net ALARMB: track 2.11 -> 1.55 mm

Commit message: almost fully routed
Parts:
- removed AND_IC2: SN74AUP1G08QDCKRQ1, SamacSys_Parts:SOT65P210X110-5N
- added NAND_IC: SN74LVC1G132DCKT, SamacSys_Parts:SOT65P210X110-5N
- AND_IC: value SN74ALVC08 -> SN74ALVC08LARGE; device SamacSys_Parts:SN74ALVC08 -> SamacSys_Parts:SN74LVC86ARGYR
- moved AND_IC 14.0 mm to (3.17, 12.2), turned to 180 degrees
- moved R12 11.1 mm to (13.4, -2.95)
- moved L2 10.1 mm to (15.7, -2.90), turned to 270 degrees
- moved XOR_IC 9.99 mm to (3.80, 6.60)
- moved R1 5.72 mm to (6.05, 12.2), turned to 90 degrees
- moved L3 3.86 mm to (6.50, 9.45), turned to 270 degrees
- moved L1 2.73 mm to (18.6, 14.5), turned to 90 degrees
- moved C12 2.60 mm to (8.10, 10.1)
- moved C11 1.40 mm to (10.1, 11.4)
- moved R15 1.30 mm to (8.90, 11.7)
- moved R7 1.22 mm to (19.4, 13.0)
- moved R14 1.22 mm to (7.70, 11.9)
- moved U1 1.00 mm to (13.6, 10.1)
- moved C16 0.85 mm to (17.2, 11.9)
- moved C9 0.81 mm to (18.4, 8.25)
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Connections:
- removed net GPIO2: J1.17, J2.2
- net A0: now also AND_IC.12, J1.16, XOR_IC.10; no longer AND_IC.1, J1.11, XOR_IC.2
- net A1: now also AND_IC.9, J1.14, XOR_IC.13; no longer AND_IC.4, J1.13, XOR_IC.5
- net A2: now also AND_IC.4, J1.13, XOR_IC.2; no longer AND_IC.8, J1.14, XOR_IC.9
- net A3: now also J1.11, NAND_IC.1, XOR_IC.5; no longer AND_IC.11, J1.16, XOR_IC.12
- net CS: now also AND_IC.1, NAND_IC.4; no longer AND_IC.13, AND_IC2.1
- net GND: now also AND_IC.15, NAND_IC.3, XOR_IC.15; no longer AND_IC2.3
- net GPIO1: now also AND_IC.2, J1.17, J2.2; no longer AND_IC2.2
- net IN5: now also J1.18, J2.1
- net IN6: no longer J1.18, J2.1
- net N$11: now also AND_IC.10, AND_IC.11, XOR_IC.12; no longer AND_IC.3, AND_IC.5, XOR_IC.4
- net N$13: now also AND_IC.5, AND_IC.8, XOR_IC.1; no longer AND_IC.6, AND_IC.9, XOR_IC.8
- net N$16: now also AND_IC.6, NAND_IC.2, XOR_IC.4; no longer AND_IC.10, AND_IC.12, XOR_IC.11
- net N$5: now also AND_IC.3; no longer AND_IC2.4
- net S0: now also J2.3, XOR_IC.8; no longer J2.8, XOR_IC.3
- net S1: now also J2.5, XOR_IC.11; no longer J2.6, XOR_IC.6
- net S2: now also J2.6, XOR_IC.3; no longer J2.5, XOR_IC.10
- net S3: now also J2.8, XOR_IC.6; no longer J2.3, XOR_IC.13
- net VDD: now also AND_IC.13, NAND_IC.5, XOR_IC.9; no longer AND_IC.2, AND_IC2.5, XOR_IC.1
Routing:
- net A2: track 0.00 -> 28.4 mm
- net IN6: track 33.1 -> 11.2 mm, vias 2 -> 1
- net S2: track 0.00 -> 21.9 mm, vias 0 -> 2
- net A1: track 0.00 -> 20.0 mm, vias 0 -> 2
- net N$16: track 0.00 -> 19.5 mm, vias 0 -> 1
- net SCLK: track 4.39 -> 21.6 mm, vias 0 -> 2
- net GPIO2: track 16.6 -> 0.00 mm, vias 2 -> 0
- net GPIO1: track 0.00 -> 16.6 mm, vias 0 -> 2
- net S3: track 0.00 -> 16.0 mm, vias 0 -> 2
- net IN5: track 10.2 -> 25.4 mm, vias 1 -> 2
- net A0: track 0.00 -> 14.4 mm, vias 0 -> 2
- net CS: track 1.48 -> 14.8 mm
- net S1: track 0.00 -> 13.3 mm, vias 0 -> 2
- net VDD: track 46.6 -> 33.6 mm, vias 2 -> 1
- net N$13: track 0.00 -> 12.6 mm
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- added copper zone on layer 16, net IN6
- removed copper zone on layer 16, net IN5

Commit message: ready for prod
Parts:
- moved R12 13.1 mm to (6.75, 8.30)
- moved L2 12.7 mm to (9.46, 8.20)
- moved C12 1.42 mm to (9.45, 9.60)
- moved L3 0.63 mm to (6.20, 10.0), turned to 180 degrees
- moved U$1 0.35 mm to (17.5, 5.64)
- moved C11 0.34 mm to (9.95, 11.7)
- moved C13 0.28 mm to (19.3, 5.00)
- moved NAND_IC 0.25 mm to (10.1, 5.60)
- moved R14 0.25 mm to (7.70, 12.2)
- moved R15 0.25 mm to (8.90, 11.9)
- moved AND_IC 0.16 mm to (3.23, 12.1)
Routing:
- net VDD: track 33.6 -> 69.2 mm, vias 1 -> 2
- net GND: track 28.4 -> 54.7 mm, vias 4 -> 14
- net GPIO1: track 16.6 -> 25.1 mm
- net S2: track 21.9 -> 24.9 mm
- net SYNCB: track 21.2 -> 23.7 mm
- net A2: track 28.4 -> 30.4 mm
- net N$16: track 19.5 -> 21.5 mm, vias 1 -> 2
- net N$13: track 12.6 -> 10.9 mm
- net A0: track 14.4 -> 12.8 mm
- net N$6: track 0.00 -> 1.50 mm
- net RLDREF: track 2.95 -> 1.79 mm
- net N$7: track 0.00 -> 1.04 mm
- net N$2: track 0.00 -> 0.97 mm
- net IN6: track 11.2 -> 12.1 mm
- net S3: track 16.0 -> 17.0 mm
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Other:
- board text added: "ads1293-v2.1"
- board text removed: "ads1293-4l-fpc-v12"
