File: master/clvHd_Master.sch (EAGLE design)
At the start: 33 parts, among them IC1 ATSAMD21J18A-MUT, IC2 RT9080-33GJ5, J1 XF2J-1024-12, J3 XF2J-1024-12, J4 MICRO-SDFRICTION, X1 BM02B-SRSS-TB, X21 BM10B-SRSS-TB, X22 BM10B-SRSS-TB, X23 BM10B-SRSS-TB, X24 BM10B-SRSS-TB

Commit message: master update
Parts:
- removed X21, X22, X23, X24: BM10B-SRSS-TB, con-JST SH:BM10B-SRSS-TB
- added X3: 1501_04, con-lumberg:1501_04
- J1: value XF2J-1024-12 -> XF2J-1824-12; device con-omron:XF2J-1024-12 -> con-omron:XF2J-1824-12
Connections:
- removed net CS1: X21.1
- removed net CS10: X22.9
- removed net CS11: X23.1
- removed net CS12: X23.3
- removed net CS13: X23.5
- removed net CS14: X23.7
- removed net CS15: X23.9
- removed net CS16: X24.1
- removed net CS17: X24.3
- removed net CS18: X24.5
- removed net CS19: X24.7
- removed net CS2: X21.3
- removed net CS20: X24.9
- removed net CS3: X21.5
- removed net CS4: X21.7
- removed net CS5: X21.9
- removed net CS6: X22.1
- removed net CS7: X22.3
- removed net CS8: X22.5
- removed net CS9: X22.7
- removed net D1: X21.2
- removed net D10: X22.10
- removed net D11: X23.2
- removed net D12: X23.4
- removed net D13: X23.6
- removed net D14: X23.8
- removed net D15: X23.10
- removed net D16: X24.2
- removed net D17: X24.4
- removed net D18: X24.6
- removed net D19: X24.8
- removed net D2: X21.4
- removed net D20: X24.10
- removed net D3: X21.6
- removed net D4: X21.8
- removed net D5: X21.10
- removed net D6: X22.2
- removed net D7: X22.4
- removed net D8: X22.6
- removed net D9: X22.8
Other:
- moved on the sheet: J1-1, J1-10, J1-2, J1-3, J1-4, J1-5, J1-6, J1-7, J1-8, J1-9, J3-1, J3-10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
