File: KiCad/ADS1293/hc32l110/ext_board_drv2605/ext_board_drv2605.kicad_sch (KiCad schematic)
At the start: 15 parts, among them J0 Conn_01x02_Male, J11 Conn_01x01_Female, J12 Conn_01x01_Female, J13 Conn_01x01_Female, J21 Conn_01x01_Female, J22 Conn_01x01_Female, J23 Conn_01x01_Female, J31 Conn_01x01_Female, J32 Conn_01x01_Female, J33 Conn_01x01_Female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

Commit message: updated
Parts:
- removed J33: Conn_01x01_Female, 00_Custom:Pin_D1.2mm_pogo, symbol Connector:Conn_01x01_Female
- removed U1: DRV2605YZFR, 00_Custom:DSBGA-9, symbol custom:DRV2605YZFR
- added M1: LRA, 00_Custom:LRA0832BE03L15, symbol custom:Actuator
- added U1: DRV2605L, 00_Custom:DRV2605L-VSSOP, symbol custom:DRV2605L
- added U2: WS2812-2020, 00_Custom:WS2812-2020, symbol custom:WS2812-2020
- J0: footprint (none) -> Connector_PinHeader_1.00mm:PinHeader_1x02_P1.00mm_Vertical
Connections:
- net +3.3V: now also U1.10 (VDD), U1.6 (VDD/NC), U2.4 (VDD)
- net GND: now also U1.8 (GND), U2.2 (GND)
- net I2C_SCL: now also U1.2 (SCL)
- net I2C_SDA: now also U1.3 (SDA)
- net OUT1: now also U1.4 (IN/TRIG)
- net OUT2: now also U2.3 (DI)
- net OUT3: now also U1.5 (EN)
- net reg: now reaches C1.1
- net reg: now also U1.1 (REG)
- net MOT-: now reaches J0.2 (Pin_2)
- net MOT-: now also U1.9 (OUT-)
- net MOT+: now reaches J0.1 (Pin_1)
- net MOT+: now also U1.7 (OUT+)
- no-connect marks 0 -> 1
Other:
- moved on the sheet: C1, J0

Commit message: updated
Parts:
- M1: footprint 00_Custom:LRA0832BE03L15 -> 00_custom-footprints:LRA0832BE03L15
- U1: footprint 00_Custom:DRV2605L-VSSOP -> 00_custom-footprints:DRV2605L-VSSOP
- U2: footprint 00_Custom:WS2812-2020 -> 00_custom-footprints:WS2812-2020
Other:
- moved on the sheet: C1, J0, J11, J12, J13, J21, J22, J23, J31, J32, J41, J42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
