File: KiCad/ADS1293/ads1293_logic_add/ads1293_logic_add.kicad_pcb (KiCad board)
At the start: 8 copper layers, 23 x 19 mm, 24 parts, among them J1 COM_IN, J2 COM_OUT, U1 ADS1293CISQE-NOPB, U2 SN74LVC1G132DCKR, U3 SN74ALVC08RGYR, U4 SN74LVC86ARGYR

Commit message: lot of modification, preparing a refactor + some rendering
Parts:
- removed R4: 51, Capacitor_SMD:C_0201_0603Metric
- removed TP1: TP_SDA, 00_Custom:TestPoint_Pad_D1.0mm
- removed TP2: TP_SCL, 00_Custom:TestPoint_Pad_D1.0mm
- removed TP4: TP_AUX2, 00_Custom:TestPoint_Pad_D1.0mm
- added C7: 100nF, Capacitor_SMD:C_0402_1005Metric, F.Cu at (191.1, 98.5)
- added C8: 100nF, Capacitor_SMD:C_0402_1005Metric, F.Cu at (196.6, 101.3)
- added I1: smd_insert, 00_custom-footprints:insert_1.2mm, F.Cu at (181.5, 105.0)
- added I2: smd_insert, 00_custom-footprints:insert_1.2mm, F.Cu at (199.5, 105.0)
- added I3: smd_insert, 00_custom-footprints:insert_1.2mm, F.Cu at (199.5, 90.5)
- added I4: smd_insert, 00_custom-footprints:insert_1.2mm, F.Cu at (181.5, 90.5)
- added TP10: TP_SDA, 00_custom-footprints:TestPoint_Pad_D1.0mm, F.Cu at (182.5, 102.0)
- added TP11: TP_AUX2, 00_custom-footprints:TestPoint_Pad_D1.0mm, F.Cu at (199.5, 93.5)
- added TP8: TP_AUX3, 00_custom-footprints:TestPoint_Pad_D1.0mm, F.Cu at (199.6, 95.5)
- added kibuzzard-63F61033: G***, kibuzzard-63F61033, F.Cu at (180.5, 99.0)
- C1, C2, C5, C6, R1, R2: footprint Capacitor_SMD:C_0201_0603Metric -> Capacitor_SMD:C_0402_1005Metric
- C3: value 1uF -> 100nF; footprint Capacitor_SMD:C_0201_0603Metric -> Capacitor_SMD:C_0402_1005Metric
- C4: value 100nF -> 1uF; footprint Capacitor_SMD:C_0201_0603Metric -> Capacitor_SMD:C_0402_1005Metric
- J1: value COM_IN -> XF2J-1824-12A; footprint 00_Custom:XF2J-1824-12A -> 00_custom-footprints:XF2J-1824-12A
- J2: value COM_OUT -> XF2J-1824-12A; footprint 00_Custom:XF2J-1824-12A -> 00_custom-footprints:XF2J-1824-12A
- LED1: footprint 00_Custom:WS2812-2020 -> 00_custom-footprints:WS2812-2020
- R3: value 1M -> 51; footprint Capacitor_SMD:C_0201_0603Metric -> Capacitor_SMD:C_0402_1005Metric
- TP5: value TP_AUX3 -> TP_SCL; footprint 00_Custom:TestPoint_Pad_D1.0mm -> 00_custom-footprints:TestPoint_Pad_D1.0mm
- TP6: renamed from TP3; value TP_AUX1 -> TP_CS
- TP6: value TP_CS -> TP_AUX1; footprint 00_Custom:TestPoint_Pad_D1.0mm -> 00_custom-footprints:TestPoint_Pad_D1.0mm
- U1: footprint 00_Custom:ADS1293CISQE -> 00_custom-footprints:ADS1293CISQE
- U2: footprint 00_Custom:SN74LVC1G132DCKR -> 00_custom-footprints:SN74LVC1G132DCKR
- U3: value SN74ALVC08RGYR -> SN74LVC86ARGYR; footprint 00_Custom:SN74ALVC08RGYR -> 00_custom-footprints:SN74LVC86ARGYR
- U4: value SN74LVC86ARGYR -> SN74ALVC08RGYR; footprint 00_Custom:SN74LVC86ARGYR -> 00_custom-footprints:SN74ALVC08RGYR
- XTAL1: footprint 00_Custom:SMD3225-4P -> 00_custom-footprints:SMD3225-4P
- moved TP6 65.8 mm to (197.7, 94.3)
- moved TP5 54.3 mm to (188.5, 95.5)
- moved TP6 53.9 mm to (190.5, 100.5)
- moved C5 33.5 mm to (196.8, 102.4), turned to 0 degrees
- moved J1 32.9 mm to (190.5, 104.0)
- moved LED1 31.2 mm to (182.1, 94.4)
- moved C4 29.1 mm to (199.2, 96.6)
- moved C6 28.4 mm to (190.7, 96.1)
- moved U1 28.2 mm to (194.4, 98.0)
- moved R2 28.1 mm to (190.7, 97.0)
- moved C3 27.9 mm to (197.8, 95.9), turned to -90 degrees
- moved XTAL1 27.8 mm to (198.9, 99.9)
- moved R1 27.7 mm to (190.1, 95.1)
- moved C2 27.4 mm to (198.9, 102.3), turned to 0 degrees
- moved C1 27.0 mm to (198.4, 97.6)
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Connections:
- net /carry0 renamed /logic_address_unit/carry0
- net /carry1 renamed /logic_address_unit/carry1
- net /carry2 renamed /logic_address_unit/carry2
- net Net-(C6-Pad1) renamed /ADS1293CISQE_0402_unit/RLDINV
- net Net-(C6-Pad2) renamed /ADS1293CISQE_0402_unit/RLDOUT
- net Net-(R1-Pad2) renamed /ADS1293CISQE_0402_unit/CMOUT
- C3 pad 1: Net-(C3-Pad1) -> +5VA
- C4 pad 1: +3.3V -> /ADS1293CISQE_0402_unit/cvref
- C5 pad 1: Net-(C5-Pad1) -> +3.3V
- J1 pad 1: IN_ref -> LED_IN
- J1 pad 12: AUX2 -> SCLK
- J1 pad 13: AUX3 -> AUX2
- J1 pad 14: SCLK -> DIN
- J1 pad 15: DIN -> GND
- J1 pad 17: GND -> +5VA
- J1 pad 2: GND -> ADD_IN1
- J1 pad 3: LED_IN -> ADD_IN2
- J1 pad 4: ADD_IN1 -> ADD_IN3
- J1 pad 5: I2C_SDA -> ADD_IN4
- J1 pad 6: I2C_SCL -> I2C_SDA
- J1 pad 7: ADD_IN2 -> I2C_SCL
- J1 pad 8: ADD_IN3 -> AUX3
- J1 pad 9: ADD_IN4 -> IN_ref
- J2 pad 10: ADD_OUT4 -> IN_ref
- J2 pad 11: ADD_OUT3 -> AUX3
- J2 pad 12: ADD_OUT2 -> I2C_SCL
- J2 pad 13: I2C_SCL -> I2C_SDA
- J2 pad 14: I2C_SDA -> ADD_OUT4
- J2 pad 15: ADD_OUT1 -> ADD_OUT3
- J2 pad 16: LED_OUT -> ADD_OUT2
- J2 pad 17: GND -> ADD_OUT1
- J2 pad 18: IN_ref -> LED_OUT
- J2 pad 2: GND -> +5VA
- J2 pad 4: DIN -> GND
- J2 pad 5: SCLK -> DIN
- J2 pad 6: AUX3 -> AUX2
- J2 pad 7: AUX2 -> SCLK
- R3 pad 1: /drdy -> (no net)
- R3 pad 2: +3.3V -> DOUT
- TP5 pad 1: AUX3 -> I2C_SCL
- TP6 pad 1: AUX1 -> CSB
- TP6 pad 1: CS -> AUX1
- U1 pad 11: Net-(C5-Pad1) -> /ADS1293CISQE_0402_unit/RLDREF
- U1 pad 12: Net-(C5-Pad1) -> /ADS1293CISQE_0402_unit/RLDREF
- U1 pad 15: unconnected-(U1-Pad15) -> /ADS1293CISQE_0402_unit/ALARMB
- U1 pad 16: CS -> CSB
- U1 pad 19: Net-(R4-Pad1) -> /ADS1293CISQE_0402_unit/sdo
- U1 pad 20: /drdy -> /ADS1293CISQE_0402_unit/D_RDYB
- U1 pad 22: unconnected-(U1-Pad22) -> +3.3V
- U1 pad 26: Net-(C3-Pad1) -> /ADS1293CISQE_0402_unit/cvref
- U1 pad 28: +3.3V -> +5VA
- U2 pad 2: /A3 -> ADD_IN4
- U2 pad 4: unconnected-(U2-Pad4) -> CSB
- U3 pad 1: /A1 -> ADD_IN2
- U3 pad 11: /S2 -> ADD_OUT3
- U3 pad 12: /A2 -> ADD_IN3
- U3 pad 3: /S1 -> ADD_OUT2
- U3 pad 4: /A0 -> ADD_IN1
- U3 pad 6: /S0 -> ADD_OUT1
- U3 pad 8: /S3 -> ADD_OUT4
- U3 pad 9: /A3 -> ADD_IN4
- U4 pad 10: /A2 -> ADD_IN3
- U4 pad 2: /A0 -> ADD_IN1
- U4 pad 5: /A1 -> ADD_IN2
Routing:
- net +5VA: track 0.00 -> 36.8 mm
- net I2C_SCL: track 0.00 -> 36.5 mm, vias 0 -> 2
- net AUX2: track 1.05 -> 36.2 mm, vias 1 -> 3
- net DIN: track 3.94 -> 37.5 mm, vias 0 -> 2
- net AUX1: track 7.29 -> 40.7 mm, vias 0 -> 3
- net AUX3: track 3.43 -> 35.8 mm, vias 0 -> 2
- net SCLK: track 6.33 -> 38.0 mm, vias 0 -> 2
- net I2C_SDA: track 5.56 -> 34.2 mm, vias 1 -> 3
- net DOUT: track 9.47 -> 34.1 mm, vias 0 -> 2
- net IN_ref: track 37.2 -> 16.4 mm
- net /A2: track 14.0 -> 0.00 mm
- net /logic_address_unit/carry1: track 12.4 -> 0.00 mm
- net unconnected-(J1-sh1-Pad19): track 10.3 -> 0.00 mm, vias 1 -> 0
- net ADD_OUT3: track 0.00 -> 7.18 mm
- net ADD_OUT1: track 0.00 -> 7.09 mm
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- added copper zone on B.Cu, net IN1
- added copper zone on B.Cu, net IN2
- added copper zone on B.Cu, net IN3
- added copper zone on B.Cu, net IN4
- added copper zone on B.Cu, net IN5
Other:
- board size 23 x 19 mm -> 22 x 18.5 mm
- copper layers 8 -> 4
- board text added: "1"
- board text added: "5"
- board text added: "ClvHd-v2.9"
