File: KiCad/ADS1293/ads1293_logic_add/ads1293_logic_add.kicad_sch (KiCad schematic)
At the start: 24 parts, among them J1 COM_IN, J2 COM_OUT, U1 ADS1293CISQE-NOPB, U2 SN74LVC1G132DCKR, U3 SN74ALVC08RGYR, U4 SN74LVC86ARGYR

Commit message: lot of modification, preparing a refactor + some rendering
Parts:
- removed C1, C2: 22pF, Capacitor_SMD:C_0201_0603Metric, symbol Device:C
- removed C3: 1uF, Capacitor_SMD:C_0201_0603Metric, symbol Device:C
- removed C4, C5: 100nF, Capacitor_SMD:C_0201_0603Metric, symbol Device:C
- removed C6: 1nF, Capacitor_SMD:C_0201_0603Metric, symbol Device:C
- removed J1: COM_IN, 00_Custom:XF2J-1824-12A, symbol XF2J-1824-12A:XF2J-1824-12A
- removed J2: COM_OUT, 00_Custom:XF2J-1824-12A, symbol XF2J-1824-12A:XF2J-1824-12A
- removed R1: 10K, Capacitor_SMD:C_0201_0603Metric, symbol Device:R
- removed R2: 10M, Capacitor_SMD:C_0201_0603Metric, symbol Device:R
- removed R3: 1M, Capacitor_SMD:C_0201_0603Metric, symbol Device:R
- removed R4: 51, Capacitor_SMD:C_0201_0603Metric, symbol Device:R
- removed U1: ADS1293CISQE-NOPB, 00_Custom:ADS1293CISQE, symbol ads1293:ADS1293CISQE-NOPB
- removed U2: SN74LVC1G132DCKR, 00_Custom:SN74LVC1G132DCKR, symbol SN74LVC1G132DCKR:SN74LVC1G132DCKR
- removed U3: SN74ALVC08RGYR, 00_Custom:SN74ALVC08RGYR, symbol SN74ALVC08RGYR:SN74ALVC08RGYR
- removed U4: SN74LVC86ARGYR, 00_Custom:SN74LVC86ARGYR, symbol SN74LVC86ARGYR:SN74LVC86ARGYR
- removed XTAL1: 4.096MHz, 00_Custom:SMD3225-4P, symbol custom:XTAL
- LED1, TP1, TP2, TP3, TP4, TP5, TP6: now left out of the parts list
Connections:
- net CS renamed CSB
- no-connect marks 7 -> 0
Other:
- added sheet ADS1293CISQE_0402_unit (ADS1293CISQE_0402_unit.kicad_sch)
- added sheet comBusIN_v2 (comBusIN_v2.kicad_sch)
- added sheet comBusOUT_v2 (comBusOUT_v2.kicad_sch)
- added sheet logic_address_unit (logic_address_unit.kicad_sch)
