File: KiCad/ADS1293/hc32l110/hc32l110.kicad_pcb (KiCad board)
At the start: 4 copper layers, 22 x 18.5 mm, 30 parts, among them J1 COM_IN, J2 COM_OUT, U1 ADS1293CISQE-NOPB, U2 HC32L110C6UA

Commit message: updated
Parts:
- added I1: smd_insert, 00_Custom:insert_1.2mm, F.Cu at (169.4, 91.5)
- added I2: smd_insert, 00_Custom:insert_1.2mm, F.Cu at (187.4, 91.5)
- added I3: smd_insert, 00_Custom:insert_1.2mm, F.Cu at (187.4, 77.0)
- added I4: smd_insert, 00_Custom:insert_1.2mm, F.Cu at (169.4, 77.0)
Changed lines of the file:
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@@
   (net 49 "RESETB")
   (net 50 "AUX2")
+  (net 51 "unconnected-(I1-Pad1)")
+  (net 52 "unconnected-(I2-Pad1)")
+  (net 53 "unconnected-(I3-Pad1)")
+  (net 54 "unconnected-(I4-Pad1)")
   (footprint "Capacitor_SMD:C_0201_0603Metric" (layer "F.Cu")
     (at 178.61 82.755)
@@
       ) (layer "F.SilkS") (width 0) (fill solid))
   )
+  (footprint "00_Custom:insert_1.2mm" (layer "F.Cu")
+    (at 169.38 76.98)
+    (property "Sheetfile" "hc32l110.kicad_sch")
+    (property "Sheetname" "")
+    (attr smd)
+    (fp_text reference "I4" (at 0 -0.05 unlocked) (layer "F.SilkS") hide
+      (effects (font (size 1 1) (thickness 0.15)))
+    )
+    (fp_text value "smd_insert" (at 0 0 unlocked) (layer "F.Fab") hide
+      (effects (font (size 1 0.2) (thickness 0.05)))
+    )
+    (fp_text user "${REFERENCE}" (at 0 -0.05 unlocked) (layer "F.Fab") hide
+      (effects (font (size 1 1) (thickness 0.15)))
+    )
+    (pad "1" smd circle (at 0 0) (size 3 3) (layers "F.Cu" "F.Mask")
+      (net 54 "unconnected-(I4-Pad1)") (pinfunction "conn") (pintype "power_in") (solder_mask_margin -0.5))
+    (model "/home/aightech/KICAD/libs/custom_lib/step/insert_2mm.step"
+      (offset (xyz 0 0 0))
+      (scale (xyz 1 1 1))
+      (rotate (xyz 0 0 0))
+    )
+  )
   (footprint "Capacitor_SMD:C_0201_0603Metric" (layer "F.Cu")
     (at 186.32 84.61 180)
@@
     (pad "1" smd circle (at 0 0) (size 1 1) (layers "F.Cu" "F.Mask")
       (net 41 "OUT1") (pinfunction "1") (pintype "passive"))
+  )
+  (footprint "00_Custom:insert_1.2mm" (layer "F.Cu")
+    (at 187.38 91.48)
+    (property "Sheetfile" "hc32l110.kicad_sch")
+    (property "Sheetname" "")
+    (attr smd)
+    (fp_text reference "I2" (at 0 -0.05 unlocked) (layer "F.SilkS") hide
+      (effects (font (size 1 1) (thickness 0.15)))
+    )
+    (fp_text value "smd_insert" (at 0 0 unlocked) (layer "F.Fab") hide
+      (effects (font (size 1 0.2) (thickness 0.05)))
+    )
+    (fp_text user "${REFERENCE}" (at 0 -0.05 unlocked) (layer "F.Fab") hide
+      (effects (font (size 1 1) (thickness 0.15)))
+    )
+    (pad "1" smd circle (at 0 0) (size 3 3) (layers "F.Cu" "F.Mask")
+      (net 52 "unconnected-(I2-Pad1)") (pinfunction "conn") (pintype "power_in") (solder_mask_margin -0.5))
+    (model "/home/aightech/KICAD/libs/custom_lib/step/insert_2mm.step"
+      (offset (xyz 0 0 0))
+      (scale (xyz 1 1 1))
+      (rotate (xyz 0 0 0))
+    )
   )
   (footprint "00_Custom:WS2812-2020" (layer "F.Cu")
@@
     )
   )
+  (footprint "00_Custom:insert_1.2mm" (layer "F.Cu")
+    (at 187.38 76.98)
+    (property "Sheetfile" "hc32l110.kicad_sch")
+    (property "Sheetname" "")
+    (attr smd)
+    (fp_text reference "I3" (at 0 -0.05 unlocked) (layer "F.SilkS") hide
+      (effects (font (size 1 1) (thickness 0.15)))
+    )
+    (fp_text value "smd_insert" (at 0 0 unlocked) (layer "F.Fab") hide
+      (effects (font (size 1 0.2) (thickness 0.05)))
+    )
+    (fp_text user "${REFERENCE}" (at 0 -0.05 unlocked) (layer "F.Fab") hide
+      (effects (font (size 1 1) (thickness 0.15)))
+    )
+    (pad "1" smd circle (at 0 0) (size 3 3) (layers "F.Cu" "F.Mask")
+      (net 53 "unconnected-(I3-Pad1)") (pinfunction "conn") (pintype "power_in") (solder_mask_margin -0.5))
+    (model "/home/aightech/KICAD/libs/custom_lib/step/insert_2mm.step"
+      (offset (xyz 0 0 0))
+      (scale (xyz 1 1 1))
+      (rotate (xyz 0 0 0))
+    )
+  )
   (footprint "00_Custom:TestPoint_Pad_D1.0mm" (layer "F.Cu")
     (at 187.38 82.98)
@@
     (pad "1" smd circle (at 0 0) (size 1 1) (layers "F.Cu" "F.Mask")
       (net 50 "AUX2") (pinfunction "1") (pintype "passive"))
+  )
+  (footprint "00_Custom:insert_1.2mm" (layer "F.Cu")
+    (at 169.38 91.48)
+    (property "Sheetfile" "hc32l110.kicad_sch")
+    (property "Sheetname" "")
+    (attr smd)
+    (fp_text reference "I1" (at 0 -0.05 unlocked) (layer "F.SilkS") hide
+      (effects (font (size 1 1) (thickness 0.15)))
+    )
+    (fp_text value "smd_insert" (at 0 0 unlocked) (layer "F.Fab") hide
+      (effects (font (size 1 0.2) (thickness 0.05)))
+    )
+    (fp_text user "${REFERENCE}" (at 0 -0.05 unlocked) (layer "F.Fab") hide
+      (effects (font (size 1 1) (thickness 0.15)))
+    )
+    (pad "1" smd circle (at 0 0) (size 3 3) (layers "F.Cu" "F.Mask")
+      (net 51 "unconnected-(I1-Pad1)") (pinfunction "conn") (pintype "power_in") (solder_mask_margin -0.5))
+    (model "/home/aightech/KICAD/libs/custom_lib/step/insert_2mm.step"
+      (offset (xyz 0 0 0))
+      (scale (xyz 1 1 1))
+      (rotate (xyz 0 0 0))
+    )
   )
   (footprint "Capacitor_SMD:C_0201_0603Metric" (layer "F.Cu")
@@
     )
   )
-  (gr_circle (center 169.379999 76.979999) (end 170.879999 76.979999) (layer "F.Cu") (width 0) (fill solid))
-  (gr_circle (center 169.38 91.48) (end 170.88 91.48) (layer "F.Cu") (width 0) (fill solid))
-  (gr_circle (center 187.38 91.48) (end 188.88 91.48) (layer "F.Cu") (width 0) (fill solid))
-  (gr_circle (center 187.379999 76.979999) (end 188.879999 76.979999) (layer "F.Cu") (width 0) (fill solid))
   (gr_poly
     (pts
@@
   (gr_circle (center 185.88 77.48) (end 187.38 77.48) (layer "B.Mask") (width 0) (fill solid))
   (gr_rect (start 184.38 77.48) (end 187.38 90.98) (layer "B.Mask") (width 0) (fill solid))
-  (gr_circle (center 187.379999 76.979999) (end 188.379999 76.979999) (layer "F.Mask") (width 0) (fill solid))
-  (gr_circle (center 187.38 91.48) (end 188.38 91.48) (layer "F.Mask") (width 0) (fill solid))
-  (gr_circle (center 169.38 91.48) (end 170.38 91.48) (layer "F.Mask") (width 0) (fill solid))
-  (gr_circle (center 169.379999 76.979999) (end 170.379999 76.979999) (layer "F.Mask") (width 0) (fill solid))
   (gr_arc (start 169.38 93.48) (mid 167.965786 92.894214) (end 167.38 91.48) (layer "Edge.Cuts") (width 0.1))
   (gr_line (start 169.379999 74.979999) (end 187.379999 74.979999) (layer "Edge.Cuts") (width 0.1))
@@
   (segment (start 182.829999 87.760001) (end 182.829999 86.88) (width 0.127) (layer "F.Cu") (net 45))
   (segment (start 182.74 87.85) (end 182.829999 87.760001) (width 0.127) (layer "F.Cu") (net 45))
-  (segment (start 188.46 81.06) (end 187.38 79.98) (width 0.127) (layer "F.Cu") (net 46))
+  (segment (start 187.34 89.02) (end 187.717958 89.02) (width 0.127) (layer "F.Cu") (net 46))
   (segment (start 187.717958 89.02) (end 188.46 88.277958) (width 0.127) (layer "F.Cu") (net 46))
   (segment (start 184.331278 80.8665) (end 184.6 81.135222) (width 0.127) (layer "F.Cu") (net 46))
+  (segment (start 188.46 88.277958) (end 188.46 81.06) (width 0.127) (layer "F.Cu") (net 46))
   (segment (start 183.5465 80.8665) (end 184.331278 80.8665) (width 0.127) (layer "F.Cu") (net 46))
-  (segment (start 188.46 88.277958) (end 188.46 81.06) (width 0.127) (layer "F.Cu") (net 46))
   (segment (start 184.7365 75.8265) (end 185.32 76.41) (width 0.127) (layer "F.Cu") (net 46))
   (segment (start 185.32 76.41) (end 185.32 77.92) (width 0.127) (layer "F.Cu") (net 46))
+  (segment (start 182.13 91.68) (end 182.5335 92.0835) (width 0.127) (layer "F.Cu") (net 46))
+  (segment (start 185.53 91.76) (end 185.53 90.83) (width 0.127) (layer "F.Cu") (net 46))
+  (segment (start 188.46 81.06) (end 187.38 79.98) (width 0.127) (layer "F.Cu") (net 46))
   (segment (start 182.13 75.923) (end 182.2265 75.8265) (width 0.127) (layer "F.Cu") (net 46))
-  (segment (start 187.501597 89.02) (end 187.717958 89.02) (width 0.127) (layer "F.Cu") (net 46))
-  (segment (start 185.53 90.991597) (end 187.501597 89.02) (width 0.127) (layer "F.Cu") (net 46))
+  (segment (start 185.2065 92.0835) (end 185.53 91.76) (width 0.127) (layer "F.Cu") (net 46))
   (segment (start 184.6 81.135222) (end 184.6 82.85) (width 0.127) (layer "F.Cu") (net 46))
   (segment (start 182.2265 75.8265) (end 184.7365 75.8265) (width 0.127) (layer "F.Cu") (net 46))
   (segment (start 182.13 79.18) (end 182.13 75.923) (width 0.127) (layer "F.Cu") (net 46))
   (segment (start 185.71 82.41) (end 185.3 82.41) (width 0.127) (layer "F.Cu") (net 46))
+  (segment (start 185.53 90.83) (end 187.34 89.02) (width 0.127) (layer "F.Cu") (net 46))
   (segment (start 184.6 82.85) (end 184.73 82.98) (width 0.127) (layer "F.Cu") (net 46))
-  (segment (start 182.13 91.68) (end 182.5335 92.0835) (width 0.127) (layer "F.Cu") (net 46))
+  (segment (start 182.13 79.45) (end 183.5465 80.8665) (width 0.127) (layer "F.Cu") (net 46))
   (segment (start 182.5335 92.0835) (end 185.2065 92.0835) (width 0.127) (layer "F.Cu") (net 46))
-  (segment (start 182.13 79.45) (end 183.5465 80.8665) (width 0.127) (layer "F.Cu") (net 46))
   (segment (start 185.3 82.41) (end 184.73 82.98) (width 0.127) (layer "F.Cu") (net 46))
   (segment (start 182.13 79.18) (end 182.13 79.45) (width 0.127) (layer "F.Cu") (net 46))
-  (segment (start 185.2065 92.0835) (end 185.53 91.76) (width 0.127) (layer "F.Cu") (net 46))
   (segment (start 185.32 77.92) (end 187.38 79.98) (width 0.127) (layer "F.Cu") (net 46))
-  (segment (start 185.53 91.76) (end 185.53 90.991597) (width 0.127) (layer "F.Cu") (net 46))
   (segment (start 176.82 85.3) (end 177.4 85.3) (width 0.127) (layer "F.Cu") (net 47))
   (segment (start 178.41 86.31) (end 180.26 86.31) (width 0.127) (layer "F.Cu") (net 47))

Commit message: updated
Parts:
- J1, J2: footprint 00_Custom:XF2J-1824-12A -> 00_custom-footprints:XF2J-1824-12A
- LED1: footprint 00_Custom:WS2812-2020 -> 00_custom-footprints:WS2812-2020
- U1: footprint 00_Custom:ADS1293CISQE -> 00_custom-footprints:ADS1293CISQE
- U2: footprint 00_Custom:QFN-20-1EP_3x3mm_P0.4mm_EP1.4x1.4mm -> 00_custom-footprints:QFN-20-1EP_3x3mm_P0.4mm_EP1.4x1.4mm
- XTAL1: footprint 00_Custom:SMD3225-4P -> 00_custom-footprints:SMD3225-4P

Commit message: lot of modification, preparing a refactor + some rendering
Parts:
- J1: value COM_IN -> XF2J-1824-12A
- J2: value COM_OUT -> XF2J-1824-12A
