File: KiCad/ADS1293/hc32l110_0402/hc32l110.kicad_sch (KiCad schematic)
At the start: 33 parts, among them J1 XF2J-1824-12A, J2 XF2J-1824-12A, U1 ADS1293CISQE-NOPB, U2 HC32L110C6UA

Commit message: cleanup
Parts:
- removed C1, C2: 22pF, Capacitor_SMD:C_0402_1005Metric, symbol Device:C
- removed C3, C5, C8: 100nF, Capacitor_SMD:C_0402_1005Metric, symbol Device:C
- removed C4: 1nF, Capacitor_SMD:C_0402_1005Metric, symbol Device:C
- removed C6: 1uF, Capacitor_SMD:C_0402_1005Metric, symbol Device:C
- removed J1, J2: XF2J-1824-12A, 00_custom-footprints:XF2J-1824-12A, symbol XF2J-1824-12A:XF2J-1824-12A
- removed R1: 10K, Capacitor_SMD:C_0402_1005Metric, symbol Device:R
- removed R2: 10M, Capacitor_SMD:C_0402_1005Metric, symbol Device:R
- removed R4: 51, Capacitor_SMD:C_0402_1005Metric, symbol Device:R
- removed U1: ADS1293CISQE-NOPB, 00_custom-footprints:ADS1293CISQE, symbol ads1293:ADS1293CISQE-NOPB
- removed XTAL1: 4.096MHz, 00_custom-footprints:SMD3225-4P, symbol custom:XTAL
- TP1: value TP_CS -> TP_SDA
- renumbered C7 to C8
Connections:
- net CS renamed CSB
- no-connect marks 4 -> 0
Other:
- added sheet ADS1293CISQE_0402_unit (../../units/ADS1293CISQE_0402_unit.kicad_sch)
- added sheet comBusIN_v2 (comBusIN_v2.kicad_sch)
- added sheet comBusOUT_v2 (comBusOUT_v2.kicad_sch)
