File: KiCad/ADS1293/logicGate_hc32l110/hc32l110.kicad_pcb (KiCad board)
At the start: 8 copper layers, 22 x 18.5 mm, 24 parts, among them J1 XF2J-1824-12A, J2 XF2J-1824-12A, U1 ADS1293CISQE-NOPB, U2 HC32L110C6UA, U3 SN74ALVC08RGYR, U4 SN74LVC86ARGYR, U5 SN74LVC1G132DCKR

Commit message: updated
Parts:
- removed TP1: TP_SDA, 00_custom-footprints:TestPoint_Pad_D1.0mm
- removed U4: SN74LVC86ARGYR, 00_custom-footprints:SN74LVC86ARGYR
- removed U5: SN74LVC1G132DCKR, 00_custom-footprints:SN74LVC1G132DCKR
- removed XTAL1: 4.096MHz, 00_custom-footprints:SMD3225-4P
- added REF**: Crystal_SMD_HC49-SD, Crystal:Crystal_SMD_HC49-SD, F.Cu at (160.1, 81.0)
- U3: value SN74ALVC08RGYR -> 74HC688; footprint 00_custom-footprints:SN74ALVC08RGYR -> digikey-footprints:TSSOP-20_W4.4mm_small
- moved U3 18.8 mm to (172.4, 84.3), turned to -90 degrees
- moved LED1 7.40 mm to (177.3, 82.1), turned to 180 degrees
- moved C7 3.64 mm to (187.9, 86.5), turned to 90 degrees
- moved U2 2.62 mm to (178.0, 85.6)
- moved U1 2.34 mm to (184.7, 84.5)
- moved C3 2.30 mm to (181.4, 85.2)
- moved C4 2.30 mm to (180.9, 83.1)
- moved C8 2.30 mm to (180.6, 85.2)
- moved R1 2.30 mm to (180.9, 82.4)
- moved R2 2.30 mm to (180.9, 83.9)
- moved C5 2.22 mm to (187.9, 82.7)
- moved R3 2.21 mm to (184.7, 88.5)
- moved C6 1.86 mm to (187.9, 84.6), turned to -90 degrees
Connections:
- LED1 pad 1: LED_OUT -> unconnected-(LED1-DO-Pad1)
- LED1 pad 3: LED_IN -> unconnected-(LED1-DI-Pad3)
- U3 pad 1: +3.3V -> unconnected-(U3-G-Pad1)
- U3 pad 10: ADD_IN3 -> unconnected-(U3-GND-Pad10)
- U3 pad 14: +3.3V -> unconnected-(U3-R5-Pad14)
- U3 pad 15: GND -> unconnected-(U3-P6-Pad15)
- U3 pad 2: ADD_IN1 -> unconnected-(U3-P0-Pad2)
- U3 pad 3: /addressing/carry0 -> unconnected-(U3-R0-Pad3)
- U3 pad 4: /addressing/carry0 -> unconnected-(U3-P1-Pad4)
- U3 pad 5: ADD_IN2 -> unconnected-(U3-R1-Pad5)
- U3 pad 6: /addressing/carry1 -> unconnected-(U3-P2-Pad6)
- U3 pad 7: GND -> unconnected-(U3-R2-Pad7)
- U3 pad 8: /addressing/carry2 -> unconnected-(U3-P3-Pad8)
- U3 pad 9: /addressing/carry1 -> unconnected-(U3-R3-Pad9)
Routing:
- net +3.3V: track 45.3 -> 1.23 mm, vias 3 -> 0
- net +5VA: track 37.1 -> 1.11 mm
- net AUX1: track 35.3 -> 0.00 mm, vias 2 -> 0
- net AUX2: track 34.6 -> 0.00 mm, vias 2 -> 0
- net RESETB: track 33.9 -> 0.00 mm, vias 2 -> 0
- net I2C_SCL: track 33.4 -> 0.00 mm, vias 2 -> 0
- net I2C_SDA: track 32.8 -> 0.00 mm, vias 2 -> 0
- net GND: track 28.3 -> 6.00 mm, vias 7 -> 0
- net SCLK: track 37.8 -> 20.6 mm
- net DIN: track 37.5 -> 20.3 mm
- net IN_ref: track 16.4 -> 0.00 mm, vias 2 -> 0
- net DOUT: track 34.1 -> 17.8 mm
- net LED_IN: track 14.2 -> 0.00 mm
- net IN4: track 11.3 -> 0.00 mm, vias 2 -> 0
- net IN5: track 11.2 -> 0.00 mm, vias 2 -> 0
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- removed copper zone on B.Cu, net IN1
- removed copper zone on B.Cu, net IN2
- removed copper zone on B.Cu, net IN3
- removed copper zone on B.Cu, net IN4
- removed copper zone on B.Cu, net IN5
Other:
- copper layers 8 -> 4
- board text removed: "1"
- board text removed: "5"
