File: KiCad/archived/ADS1293/ads1293_logic_add/ads1293_logic_add.kicad_sch (KiCad schematic)
At the start: 7 parts

Commit message: renamed SPI buses
Other:
- sheet comBusIN_v2 ports: added PICO_DIN, POCI_DOUT; removed MISO_DOUT, MOSI_DIN
- sheet comBusOUT_v2 ports: added PICO_DIN, POCI_DOUT; removed MISO_DOUT, MOSI_DIN
Changed lines of the file:
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@@
       (effects (font (size 1.27 1.27)) (justify left))
     )
-    (pin "MISO_DOUT" input (at 81.28 116.84 180)
+    (pin "POCI_DOUT" input (at 81.28 116.84 180)
       (effects (font (size 1.27 1.27)) (justify left))
     )
-    (pin "MOSI_DIN" input (at 81.28 111.76 180)
+    (pin "PICO_DIN" input (at 81.28 111.76 180)
       (effects (font (size 1.27 1.27)) (justify left))
     )
@@
       (effects (font (size 1.27 1.27)) (justify right))
     )
-    (pin "MOSI_DIN" input (at 57.15 111.76 0)
+    (pin "PICO_DIN" input (at 57.15 111.76 0)
       (effects (font (size 1.27 1.27)) (justify right))
     )
-    (pin "MISO_DOUT" input (at 57.15 116.84 0)
+    (pin "POCI_DOUT" input (at 57.15 116.84 0)
       (effects (font (size 1.27 1.27)) (justify right))
     )
