File: KiCad/archived/ADS1293/logicGate_hc32l110/hc32l110.kicad_sch (KiCad schematic)
At the start: 8 parts, among them U2 HC32L110C6UA, U3 74HC688

Commit message: renamed SPI buses
Other:
- sheet comBusIN_v2 ports: added PICO_DIN, POCI_DOUT; removed MISO_DOUT, MOSI_DIN
- sheet comBusOUT_v2 ports: added PICO_DIN, POCI_DOUT; removed MISO_DOUT, MOSI_DIN
Changed lines of the file:
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@@
       (effects (font (size 1.27 1.27)) (justify right))
     )
-    (pin "MOSI_DIN" input (at 45.72 151.13 0)
+    (pin "PICO_DIN" input (at 45.72 151.13 0)
       (effects (font (size 1.27 1.27)) (justify right))
     )
-    (pin "MISO_DOUT" input (at 45.72 156.21 0)
+    (pin "POCI_DOUT" input (at 45.72 156.21 0)
       (effects (font (size 1.27 1.27)) (justify right))
     )
@@
       (effects (font (size 1.27 1.27)) (justify left))
     )
-    (pin "MISO_DOUT" input (at 69.85 156.21 180)
+    (pin "POCI_DOUT" input (at 69.85 156.21 180)
       (effects (font (size 1.27 1.27)) (justify left))
     )
-    (pin "MOSI_DIN" input (at 69.85 151.13 180)
+    (pin "PICO_DIN" input (at 69.85 151.13 180)
       (effects (font (size 1.27 1.27)) (justify left))
     )
