File: KiCad/archived/units/comBusIN_v2.kicad_sch (KiCad schematic)
At the start: 1 part, among them J1 XF2J-1824-12A

Commit message: renamed SPI buses
Connections:
- net MISO_DOUT renamed POCI_DOUT
- net MOSI_DIN renamed PICO_DIN
Changed lines of the file:
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@@
     (effects (font (size 1.27 1.27)) (justify right))
   )
-  (hierarchical_label "MISO_DOUT" (shape input) (at 113.03 116.84 180) (fields_autoplaced)
+  (hierarchical_label "POCI_DOUT" (shape input) (at 113.03 116.84 180) (fields_autoplaced)
     (effects (font (size 1.27 1.27)) (justify right))
   )
@@
     (effects (font (size 1.27 1.27)) (justify right))
   )
-  (hierarchical_label "MOSI_DIN" (shape input) (at 113.03 111.76 180) (fields_autoplaced)
+  (hierarchical_label "PICO_DIN" (shape input) (at 113.03 111.76 180) (fields_autoplaced)
     (effects (font (size 1.27 1.27)) (justify right))
   )
