File: KiCad/modules/COM_MOD/.kiri/a23af4b/COM_MOD.kicad_pcb (KiCad board)
At the start: 4 copper layers, 15 x 15.8 mm, 32 parts, among them J1 Conn_01x01_Pin, J10 XF2J-1824-12A, J11 Conn_01x01_Pin, J12 Conn_01x01_Pin, J13 Conn_01x01_Pin, J14 Conn_01x01_Pin, J15 Conn_01x01_Pin, J16 Conn_01x01_Pin, J17 Conn_01x01_Pin, J18 Conn_01x01_Pin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

Commit message: renamed SPI buses
Connections:
- net /MISO renamed /POCI
- net /MOSI renamed /PICO
- net /MOSI_ARM renamed /PICO_ARM
- net /SWDIO/MISO_ARM renamed /SWDIO/POCI_ARM
Changed lines of the file:
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@@
   (net 1 "GND")
   (net 2 "/Vcap")
-  (net 3 "/MISO")
-  (net 4 "/MOSI")
+  (net 3 "/POCI")
+  (net 4 "/PICO")
   (net 5 "unconnected-(J3-Pin_1-Pad1)")
   (net 6 "/SCLK")
@@
   (net 20 "/AUX3")
   (net 21 "/SWCLK")
-  (net 22 "/SWDIO{slash}MISO_ARM")
-  (net 23 "/MOSI_ARM")
+  (net 22 "/SWDIO{slash}POCI_ARM")
+  (net 23 "/PICO_ARM")
   (net 24 "/SCLK_ARM")
   (net 25 "/SPICS_ARM")
@@
       (stroke (width 0.1) (type solid)) (layer "F.Fab"))
     (pad "1" thru_hole rect (at 0 0) (size 1 1) (drill 0.65) (layers "*.Cu" "*.Mask")
-      (net 3 "/MISO") (pinfunction "Pin_1") (pintype "passive"))
+      (net 3 "/POCI") (pinfunction "Pin_1") (pintype "passive"))
     (model "${KICAD6_3DMODEL_DIR}/Connector_PinHeader_1.27mm.3dshapes/PinHeader_1x01_P1.27mm_Vertical.wrl"
       (offset (xyz 0 0 0))
@@
       (net 24 "/SCLK_ARM") (pinfunction "SPI_SCK") (pintype "input"))
     (pad "13" smd roundrect (at 1.45 0 180) (size 0.85 0.2) (layers "F.Cu" "F.Paste" "F.Mask") (roundrect_rratio 0.25)
-      (net 23 "/MOSI_ARM") (pinfunction "SPI_MOSI") (pintype "input"))
+      (net 23 "/PICO_ARM") (pinfunction "SPI_PICO") (pintype "input"))
     (pad "14" smd roundrect (at 1.45 -0.4 180) (size 0.85 0.2) (layers "F.Cu" "F.Paste" "F.Mask") (roundrect_rratio 0.25)
-      (net 22 "/SWDIO{slash}MISO_ARM") (pinfunction "SWDIO") (pintype "input"))
+      (net 22 "/SWDIO{slash}POCI_ARM") (pinfunction "SWDIO") (pintype "input"))
     (pad "15" smd roundrect (at 1.45 -0.8 180) (size 0.85 0.2) (layers "F.Cu" "F.Paste" "F.Mask") (roundrect_rratio 0.25)
       (net 21 "/SWCLK") (pinfunction "SWCLK") (pintype "input"))
@@
       (net 1 "GND") (pinfunction "2") (pintype "unspecified"))
     (pad "3" smd rect (at -3.25 -0.175 180) (size 0.3 1.25) (layers "F.Cu" "F.Paste" "F.Mask")
-      (net 3 "/MISO") (pinfunction "3") (pintype "unspecified"))
+      (net 3 "/POCI") (pinfunction "3") (pintype "unspecified"))
     (pad "4" smd rect (at -2.75 -0.175 180) (size 0.3 1.25) (layers "F.Cu" "F.Paste" "F.Mask")
-      (net 4 "/MOSI") (pinfunction "4") (pintype "unspecified"))
+      (net 4 "/PICO") (pinfunction "4") (pintype "unspecified"))
     (pad "5" smd rect (at -2.25 -0.175 180) (size 0.3 1.25) (layers "F.Cu" "F.Paste" "F.Mask")
       (net 6 "/SCLK") (pinfunction "5") (pintype "unspecified"))
@@
       (stroke (width 0.1) (type solid)) (layer "F.Fab"))
     (pad "1" thru_hole rect (at 0 0 180) (size 1 1) (drill 0.65) (layers "*.Cu" "*.Mask")
-      (net 22 "/SWDIO{slash}MISO_ARM") (pinfunction "Pin_1") (pintype "passive"))
+      (net 22 "/SWDIO{slash}POCI_ARM") (pinfunction "Pin_1") (pintype "passive"))
     (model "${KICAD6_3DMODEL_DIR}/Connector_PinHeader_1.27mm.3dshapes/PinHeader_1x01_P1.27mm_Vertical.wrl"
       (offset (xyz 0 0 0))
@@
       (stroke (width 0.1) (type solid)) (layer "F.Fab"))
     (pad "1" thru_hole rect (at 0 0 180) (size 1 1) (drill 0.65) (layers "*.Cu" "*.Mask")
-      (net 23 "/MOSI_ARM") (pinfunction "Pin_1") (pintype "passive"))
+      (net 23 "/PICO_ARM") (pinfunction "Pin_1") (pintype "passive"))
     (model "${KICAD6_3DMODEL_DIR}/Connector_PinHeader_1.27mm.3dshapes/PinHeader_1x01_P1.27mm_Vertical.wrl"
       (offset (xyz 0 0 0))
@@
       (stroke (width 0.1) (type solid)) (layer "F.Fab"))
     (pad "1" thru_hole rect (at 0 0) (size 1 1) (drill 0.65) (layers "*.Cu" "*.Mask")
-      (net 4 "/MOSI") (pinfunction "Pin_1") (pintype "passive"))
+      (net 4 "/PICO") (pinfunction "Pin_1") (pintype "passive"))
     (model "${KICAD6_3DMODEL_DIR}/Connector_PinHeader_1.27mm.3dshapes/PinHeader_1x01_P1.27mm_Vertical.wrl"
       (offset (xyz 0 0 0))
@@
       (net 6 "/SCLK") (pinfunction "14") (pintype "unspecified"))
     (pad "15" smd rect (at 2.75 0.175) (size 0.3 1.25) (layers "B.Cu" "B.Paste" "B.Mask")
-      (net 4 "/MOSI") (pinfunction "15") (pintype "unspecified"))
+      (net 4 "/PICO") (pinfunction "15") (pintype "unspecified"))
     (pad "16" smd rect (at 3.25 0.175) (size 0.3 1.25) (layers "B.Cu" "B.Paste" "B.Mask")
-      (net 3 "/MISO") (pinfunction "16") (pintype "unspecified"))
+      (net 3 "/POCI") (pinfunction "16") (pintype "unspecified"))
     (pad "17" smd rect (at 3.75 0.175) (size 0.3 1.25) (layers "B.Cu" "B.Paste" "B.Mask")
       (net 1 "GND") (pinfunction "17") (pintype "unspecified"))
