File: KiCad/modules/COM_MOD/.kiri/a23af4b/COM_MOD.kicad_sch (KiCad schematic)
At the start: 31 parts, among them J1 Conn_01x01_Pin, J10 XF2J-1824-12A, J11 Conn_01x01_Pin, J12 Conn_01x01_Pin, J13 Conn_01x01_Pin, J14 Conn_01x01_Pin, J15 Conn_01x01_Pin, J16 Conn_01x01_Pin, J17 Conn_01x01_Pin, J18 Conn_01x01_Pin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

Commit message: renamed SPI buses
Connections:
- net MISO renamed POCI
- net MOSI renamed PICO
- net MOSI_ARM renamed PICO_ARM
- net SWDIO/MISO_ARM renamed SWDIO/POCI_ARM
Changed lines of the file:
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@@
     (effects (font (size 1.27 1.27)) (justify right bottom))
   )
-  (label "SWDIO{slash}MISO_ARM" (at 242.57 57.15 180) (fields_autoplaced)
+  (label "SWDIO{slash}POCI_ARM" (at 242.57 57.15 180) (fields_autoplaced)
     (effects (font (size 1.27 1.27)) (justify right bottom))
   )
@@
     (effects (font (size 1.27 1.27)) (justify left bottom))
   )
-  (label "MISO" (at 77.47 60.96 0) (fields_autoplaced)
+  (label "POCI" (at 77.47 60.96 0) (fields_autoplaced)
     (effects (font (size 1.27 1.27)) (justify left bottom))
   )
@@
     (effects (font (size 1.27 1.27)) (justify right bottom))
   )
-  (label "MOSI" (at 77.47 63.5 0) (fields_autoplaced)
+  (label "PICO" (at 77.47 63.5 0) (fields_autoplaced)
     (effects (font (size 1.27 1.27)) (justify left bottom))
   )
@@
     (effects (font (size 1.27 1.27)) (justify right bottom))
   )
-  (label "MOSI_ARM" (at 115.57 138.43 180) (fields_autoplaced)
+  (label "PICO_ARM" (at 115.57 138.43 180) (fields_autoplaced)
     (effects (font (size 1.27 1.27)) (justify right bottom))
   )
@@
     (effects (font (size 1.27 1.27)) (justify right bottom))
   )
-  (label "MOSI" (at 229.87 144.78 270) (fields_autoplaced)
+  (label "PICO" (at 229.87 144.78 270) (fields_autoplaced)
     (effects (font (size 1.27 1.27)) (justify right bottom))
   )
@@
     (effects (font (size 1.27 1.27)) (justify left bottom))
   )
-  (label "MOSI_ARM" (at 242.57 59.69 180) (fields_autoplaced)
+  (label "PICO_ARM" (at 242.57 59.69 180) (fields_autoplaced)
     (effects (font (size 1.27 1.27)) (justify right bottom))
   )
@@
     (effects (font (size 1.27 1.27)) (justify left bottom))
   )
-  (label "SWDIO{slash}MISO_ARM" (at 115.57 135.89 180) (fields_autoplaced)
+  (label "SWDIO{slash}POCI_ARM" (at 115.57 135.89 180) (fields_autoplaced)
     (effects (font (size 1.27 1.27)) (justify right bottom))
   )
@@
     (effects (font (size 1.27 1.27)) (justify left bottom))
   )
-  (label "MISO" (at 227.33 144.78 270) (fields_autoplaced)
+  (label "POCI" (at 227.33 144.78 270) (fields_autoplaced)
     (effects (font (size 1.27 1.27)) (justify right bottom))
   )
@@
     (pin "11" (alternate "AIN0"))
     (pin "12" (alternate "SPI_SCK"))
-    (pin "13" (alternate "SPI_MOSI"))
+    (pin "13" (alternate "SPI_PICO"))
     (pin "14" (alternate "SWDIO"))
     (pin "15" (alternate "SWCLK"))
