File: KiCad/modules/EMG_DAQ_ADS1293/EMG_DAQ_ADS1293.kicad_sch (KiCad schematic)
At the start: 31 parts, among them J1 Conn_01x01_Pin, J10 Conn_01x01_Pin, J12 Conn_01x01_Pin, J13 Conn_01x01_Pin, J14 Conn_01x01_Pin, J15 Conn_01x01_Pin, J16 Conn_01x01_Pin, J2 Conn_01x01_Pin, J3 Conn_01x01_Pin, J4 Conn_01x01_Pin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

Commit message: refactor and fixing most of the modules
Other:
- company: (none) -> Aightech
- title: EMG DAQ ADS129 -> EMG DAQ ADS1293

Commit message: cleaned all modules + production files
Parts:
- removed U2: AP2112K-3.3TRG1, 00_custom-footprints:SOT95P285X140-5N, symbol 00_custom:AP2112K-3.3TRG1
- added U2: AP2112K-3.3TRG1, 00_lcsc:SOT-25-5_L2.9-W1.6-P0.95-LS2.8-BL, symbol 00_lcsc:AP2112K-3.3TRG1
- J1, J12, J16, J2, J3, J4, J5, J6: now not fitted; now left out of the parts list
Connections:
- net +3.3V: now also U2.1 (VIN), U2.3 (EN)
- net +3.3VA: now also U2.5 (VOUT)
- net GND: now also U2.2 (GND)
Changed lines of the file:
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@@
 	)
 	(junction
-		(at 113.03 64.77)
+		(at 113.03 62.23)
 		(diameter 0)
 		(color 0 0 0 0)
@@
 	(wire
 		(pts
-			(xy 113.03 60.96) (xy 113.03 64.77)
+			(xy 113.03 60.96) (xy 113.03 62.23)
 		)
 		(stroke
@@
 	(wire
 		(pts
-			(xy 127 69.85) (xy 127 59.69)
+			(xy 113.03 62.23) (xy 113.03 67.31)
+		)
+		(stroke
+			(width 0)
+			(type default)
+		)
+	)
+	(wire
+		(pts
+			(xy 127 64.77) (xy 127 59.69)
 		)
 		(stroke
@@
 	(wire
 		(pts
-			(xy 113.03 64.77) (xy 128.27 64.77)
+			(xy 113.03 62.23) (xy 128.27 62.23)
 		)
 		(stroke
@@
 	(wire
 		(pts
-			(xy 128.27 69.85) (xy 127 69.85)
+			(xy 128.27 64.77) (xy 127 64.77)
 		)
 		(stroke
@@
 	(wire
 		(pts
-			(xy 113.03 64.77) (xy 113.03 67.31)
-		)
-		(stroke
-			(width 0)
-			(type default)
-		)
-	)
-	(wire
-		(pts
 			(xy 166.37 134.62) (xy 171.45 134.62)
 		)
@@
 	)
 	(symbol
-		(lib_id "power:GND")
-		(at 81.28 62.23 0)
+		(lib_id "00_lcsc:AP2112K-3.3TRG1")
+		(at 140.97 62.23 0)
 		(unit 1)
 		(exclude_from_sim no)
@@
 		(on_board yes)
 		(dnp no)
-		(property "Reference" "#PWR09"
-			(at 81.28 68.58 0)
+		(fields_autoplaced yes)
+		(property "Reference" "U2"
+			(at 140.97 52.07 0)
 			(effects
 				(font
 					(size 1.27 1.27)
 				)
-				(hide yes)
 			)
 		)
-		(property "Value" "GND"
-			(at 78.74 66.04 0)
+		(property "Value" "AP2112K-3.3TRG1"
+			(at 140.97 54.61 0)
 			(effects
 				(font
@@
 			)
 		)
-		(property "Footprint" ""
-			(at 81.28 62.23 0)
+		(property "Footprint" "00_lcsc:SOT-25-5_L2.9-W1.6-P0.95-LS2.8-BL"
+			(at 140.97 72.39 0)
 			(effects
 				(font
@@
 			)
 		)
-		(property "Datasheet" ""
-			(at 81.28 62.23 0)
+		(property "Datasheet" "https://lcsc.com/product-detail/Low-Dropout-Regulators-LDO_DIODES_AP2112K-3-3TRG1_AP2112K-3-3TRG1_C51118.html"
+			(at 140.97 74.93 0)
 			(effects
 				(font
@@
 		)
 		(property "Description" ""
-			(at 81.28 62.23 0)
+			(at 140.97 62.23 0)
+			(effects
+				(font
+					(size 1.27 1.27)
+				)
+				(hide yes)
+			)
+		)
+		(property "LCSC Part" "C51118"
+			(at 140.97 77.47 0)
 			(effects
 				(font
@@
 		(pin "1"
 		)
+		(pin "5"
+		)
+		(pin "4"
+		)
+		(pin "3"
+		)
+		(pin "2"
+		)
 		(instances
-			(project "cleverhand_emgDAC"
-				(path "/0e05b0e4-5a62-483e-9fee-99ff448613b9"
-					(reference "#PWR09")
-					(unit 1)
-				)
-			)
 			(project "EMG_DAQ_ADS1293"
 				(path "/bd8cf3d8-de72-4df4-8cf2-76ef56ba4fd2"
-					(reference "#PWR07")
+					(reference "U2")
 					(unit 1)
 				)
@@
 	(symbol
 		(lib_id "power:GND")
-		(at 157.48 73.66 0)
+		(at 81.28 62.23 0)
 		(unit 1)
 		(exclude_from_sim no)
@@
 		(dnp no)
 		(property "Reference" "#PWR09"
-			(at 157.48 80.01 0)
+			(at 81.28 68.58 0)
 			(effects
 				(font
@@
 		)
 		(property "Value" "GND"
-			(at 162.56 74.93 0)
+			(at 78.74 66.04 0)
 			(effects
 				(font
@@
 		)
 		(property "Footprint" ""
-			(at 157.48 73.66 0)
+			(at 81.28 62.23 0)
 			(effects
 				(font
@@
 		)
 		(property "Datasheet" ""
-			(at 157.48 73.66 0)
+			(at 81.28 62.23 0)
 			(effects
 				(font
@@
 		)
 		(property "Description" ""
-			(at 157.48 73.66 0)
+			(at 81.28 62.23 0)
 			(effects
 				(font
@@
 			(project "EMG_DAQ_ADS1293"
 				(path "/bd8cf3d8-de72-4df4-8cf2-76ef56ba4fd2"
-					(reference "#PWR012")
+					(reference "#PWR07")
 					(unit 1)
 				)
@@
 	)
 	(symbol
-		(lib_id "00_custom:AP2112K-3.3TRG1")
-		(at 140.97 64.77 0)
+		(lib_id "power:GND")
+		(at 157.48 73.66 0)
 		(unit 1)
 		(exclude_from_sim no)
@@
 		(on_board yes)
 		(dnp no)
-		(fields_autoplaced yes)
-		(property "Reference" "U2"
-			(at 140.97 52.07 0)
-			(effects
-				(font
-					(size 1.27 1.27)
-				)
-			)
-		)
-		(property "Value" "AP2112K-3.3TRG1"
-			(at 140.97 54.61 0)
-			(effects
-				(font
-					(size 1.27 1.27)
-				)
-			)
-		)
-		(property "Footprint" "00_custom-footprints:SOT95P285X140-5N"
-			(at 139.7 83.82 0)
-			(effects
-				(font
-					(size 1.27 1.27)
-				)
-				(justify bottom)
-				(hide yes)
-			)
-		)
-		(property "Datasheet" ""
-			(at 140.97 64.77 0)
-			(effects
-				(font
-					(size 1.27 1.27)
-				)
-				(hide yes)
-			)
-		)
-		(property "Description" "\nVoltage Regulators, LDO, 600mA CMOS LDO 50mA 3.3V 250mV | Diodes Inc AP2112K-3.3TRG1\n"
-			(at 138.43 87.63 0)
-			(effects
-				(font
-					(size 1.27 1.27)
-				)
-				(justify bottom)
-				(hide yes)
-			)
-		)
-		(property "MF" "Diodes Inc."
-			(at 139.7 91.44 0)
-			(effects
-				(font
-					(size 1.27 1.27)
-				)
-				(justify bottom)
-				(hide yes)
-			)
-		)
-		(property "Package" "SOT-753 Diodes Inc."
-			(at 138.43 81.28 0)
-			(effects
-				(font
-					(size 1.27 1.27)
-				)
-				(justify bottom)
-				(hide yes)
-			)
-		)
-		(property "Price" "None"
-			(at 140.97 93.98 0)
-			(effects
-				(font
-					(size 1.27 1.27)
-				)
-				(justify bottom)
-				(hide yes)
-			)
-		)
-		(property "Check_prices" "https://www.snapeda.com/parts/AP2112K-3.3TRG1/Diodes+Inc./view-part/?ref=eda"
-			(at 138.43 87.63 0)
-			(effects
-				(font
-					(size 1.27 1.27)
-				)
-				(justify bottom)
-				(hide yes)
-			)
-		)
-		(property "PARTREV" "2-2"
-			(at 161.29 93.98 0)
-			(effects
-				(font
-					(size 1.27 1.27)
-				)
-				(justify bottom)
-				(hide yes)
-			)
-		)
-		(property "SnapEDA_Link" "https://www.snapeda.com/parts/AP2112K-3.3TRG1/Diodes+Inc./view-part/?ref=snap"
-			(at 138.43 87.63 0)
-			(effects
-				(font
-					(size 1.27 1.27)
-				)
-				(justify bottom)
-				(hide yes)
-			)
-		)
-		(property "MP" "AP2112K-3.3TRG1"
-			(at 138.43 81.28 0)
+		(property "Reference" "#PWR09"
+			(at 157.48 80.01 0)
 			(effects
 				(font
 					(size 1.27 1.27)
 				)
-				(justify bottom)
 				(hide yes)
 			)
 		)
-		(property "Purchase-URL" "https://www.snapeda.com/api/url_track_click_mouser/?unipart_id=454988&manufacturer=Diodes Inc.&part_name=AP2112K-3.3TRG1&search_term=None"
-			(at 138.43 87.63 0)
+		(property "Value" "GND"
+			(at 162.56 74.93 0)
 			(effects
 				(font
 					(size 1.27 1.27)
 				)
-				(justify bottom)
-				(hide yes)
 			)
 		)
-		(property "Availability" "In Stock"
-			(at 157.48 99.06 0)
+		(property "Footprint" ""
+			(at 157.48 73.66 0)
 			(effects
 				(font
 					(size 1.27 1.27)
 				)
-				(justify bottom)
 				(hide yes)
 			)
 		)
-		(property "MANUFACTURER" "Diodes Inc."
-			(at 140.97 96.52 0)
+		(property "Datasheet" ""
+			(at 157.48 73.66 0)
 			(effects
 				(font
 					(size 1.27 1.27)
 				)
-				(justify bottom)
 				(hide yes)
 			)
 		)
-		(property "LCSC" "C51118"
-			(at 140.97 64.77 0)
+		(property "Description" ""
+			(at 157.48 73.66 0)
 			(effects
 				(font
@@
 			)
 		)
-		(pin "5"
-		)
 		(pin "1"
 		)
-		(pin "2"
-		)
-		(pin "3"
-		)
 		(instances
+			(project "cleverhand_emgDAC"
+				(path "/0e05b0e4-5a62-483e-9fee-99ff448613b9"
+					(reference "#PWR09")
+					(unit 1)
+				)
+			)
 			(project "EMG_DAQ_ADS1293"
 				(path "/bd8cf3d8-de72-4df4-8cf2-76ef56ba4fd2"
-					(reference "U2")
+					(reference "#PWR012")
 					(unit 1)
 				)
@@
 		(unit 1)
 		(exclude_from_sim no)
-		(in_bom yes)
+		(in_bom no)
 		(on_board yes)
-		(dnp no)
+		(dnp yes)
 		(property "Reference" "J16"
 			(at 77.47 118.11 0)
@@
 		(unit 1)
 		(exclude_from_sim no)
-		(in_bom yes)
+		(in_bom no)
 		(on_board yes)
-		(dnp no)
+		(dnp yes)
 		(property "Reference" "J5"
 			(at 77.47 110.49 0)
@@
 		(unit 1)
 		(exclude_from_sim no)
-		(in_bom yes)
+		(in_bom no)
 		(on_board yes)
-		(dnp no)
+		(dnp yes)
 		(property "Reference" "J12"
 			(at 77.47 115.57 0)
@@
 		(unit 1)
 		(exclude_from_sim no)
-		(in_bom yes)
+		(in_bom no)
 		(on_board yes)
-		(dnp no)
+		(dnp yes)
 		(property "Reference" "J4"
 			(at 77.47 107.95 0)
@@
 		(unit 1)
 		(exclude_from_sim no)
-		(in_bom yes)
+		(in_bom no)
 		(on_board yes)
-		(dnp no)
+		(dnp yes)
 		(property "Reference" "J1"
 			(at 77.47 100.33 0)
@@
 		(unit 1)
 		(exclude_from_sim no)
-		(in_bom yes)
+		(in_bom no)
 		(on_board yes)
-		(dnp no)
+		(dnp yes)
 		(property "Reference" "J3"
 			(at 77.47 105.41 0)
@@
 		(unit 1)
 		(exclude_from_sim no)
-		(in_bom yes)
+		(in_bom no)
 		(on_board yes)
-		(dnp no)
+		(dnp yes)
 		(property "Reference" "J6"
 			(at 77.47 113.03 0)
@@
 		(unit 1)
 		(exclude_from_sim no)
-		(in_bom yes)
+		(in_bom no)
 		(on_board yes)
-		(dnp no)
+		(dnp yes)
 		(property "Reference" "J2"
 			(at 77.47 102.87 0)

Commit message: renamed SPI buses
Connections:
- net MISO renamed POCI
- net MOSI renamed PICO
Changed lines of the file:
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@@
 		)
 	)
-	(label "MOSI"
+	(label "PICO"
 		(at 88.9 63.5 270)
 		(fields_autoplaced yes)
@@
 		)
 	)
-	(label "MOSI"
+	(label "PICO"
 		(at 171.45 129.54 0)
 		(fields_autoplaced yes)
@@
 		)
 	)
-	(label "MISO"
+	(label "POCI"
 		(at 171.45 127 0)
 		(fields_autoplaced yes)
@@
 		)
 	)
-	(label "MISO"
+	(label "POCI"
 		(at 86.36 63.5 270)
 		(fields_autoplaced yes)
