File: KiCad/modules/IMU_ICM2094/IMU_ICM2094.kicad_pcb (KiCad board)
At the start: 4 copper layers, 15 x 11 mm, 23 parts, among them J1 Conn_01x01_Pin, J10 Conn_01x01_Pin, J11 Conn_01x01_Pin, J12 Conn_01x01_Pin, J13 Conn_01x01_Pin, J14 Conn_01x01_Pin, J7 Conn_01x01_Pin, J9 Conn_01x01_Pin, U1 MCP1700T-1802E/TT, U3 BSS138BKS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

Commit message: INA331 IMUICM
Parts:
- added J15: Conn_01x01_Pin, 00_custom-footprints:PinHeader_1x01_P1.27mm_Vertical, F.Cu at (36.6, 37.8)
- added J16: Conn_01x01_Pin, 00_custom-footprints:PinHeader_1x01_P1.27mm_Vertical, F.Cu at (31.5, 37.8)
- added J17: Conn_01x01_Pin, 00_custom-footprints:PinHeader_1x01_P1.27mm_Vertical, F.Cu at (32.8, 37.8)
- added J18: Conn_01x01_Pin, 00_custom-footprints:PinHeader_1x01_P1.27mm_Vertical, F.Cu at (31.5, 36.5)
- added J2: Conn_01x01_Pin, 00_custom-footprints:PinHeader_1x01_P1.27mm_Vertical, F.Cu at (26.8, 30.0)
- added J3: Conn_01x01_Pin, 00_custom-footprints:PinHeader_1x01_P1.27mm_Vertical, F.Cu at (28.1, 30.0)
- added J4: Conn_01x01_Pin, 00_custom-footprints:PinHeader_1x01_P1.27mm_Vertical, F.Cu at (29.4, 30.0)
- added J5: Conn_01x01_Pin, 00_custom-footprints:PinHeader_1x01_P1.27mm_Vertical, F.Cu at (30.6, 30.0)
- added J6: Conn_01x01_Pin, 00_custom-footprints:PinHeader_1x01_P1.27mm_Vertical, F.Cu at (31.9, 30.0)
- added J8: Conn_01x01_Pin, 00_custom-footprints:PinHeader_1x01_P1.27mm_Vertical, F.Cu at (34.4, 30.0)
- J1, J10, J11, J12, J13, J14, J7, J9: footprint Connector_PinHeader_1.27mm:PinHeader_1x01_P1.27mm_Vertical -> 00_custom-footprints:PinHeader_1x01_P1.27mm_Vertical
- moved J14 11.5 mm to (35.3, 37.8)
- moved J13 11.5 mm to (34.0, 37.8)
- moved J9 9.71 mm to (36.6, 36.5)
- moved J10 8.00 mm to (35.3, 36.5)
- moved J11 6.84 mm to (34.0, 36.5)
- moved J12 6.51 mm to (32.8, 36.5)
- moved R8 6.39 mm to (24.5, 38.5), turned to 0 degrees
- moved R6 6.18 mm to (24.5, 37.5), turned to 0 degrees
- moved R2 3.82 mm to (32.9, 34.4)
- moved C5 3.62 mm to (29.5, 36.7)
- moved R4 3.34 mm to (36.4, 34.4), turned to -90 degrees
- moved U4 2.87 mm to (30.0, 33.7)
- moved U5 2.87 mm to (26.9, 38.0), turned to 90 degrees
- moved J1 2.54 mm to (25.6, 30.0)
- moved C1 2.06 mm to (26.5, 31.9), turned to 0 degrees
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Connections:
- J1 pad 1: unconnected-(J1-Pin_1-Pad1) -> +3.3V
- J10 pad 1: /MOSI -> /SWDIO/MISO_ARM
- J11 pad 1: /SCLK -> /MOSI_ARM
- J12 pad 1: /CSB -> /SCLK_ARM
- J13 pad 1: +3.3V -> /SPICS_ARM
- J14 pad 1: GND -> /i2C_SCL
- J7 pad 1: /extRef -> unconnected-(J7-Pin_1-Pad1)
- J9 pad 1: /MISO -> /IO1_out
- R1 pad 2: /SCLK -> /MOSI
- R2 pad 1: /SCK_1.8V -> /MOSI_1.8V
- R3 pad 2: /CS_1.8V -> /SCK_1.8V
- R4 pad 2: /CSB -> /SCLK
- R5 pad 2: /MOSI -> /MISO
- R6 pad 1: /MOSI_1.8V -> /MISO_1.8V
- R7 pad 2: /MISO_1.8V -> /CS_1.8V
- R8 pad 2: /MISO -> /CSB
- U3 pad 1: /CS_1.8V -> /SCK_1.8V
- U3 pad 3: /SCLK -> /MOSI
- U3 pad 4: /SCK_1.8V -> /MOSI_1.8V
- U3 pad 6: /CSB -> /SCLK
- U5 pad 1: /MISO_1.8V -> /CS_1.8V
- U5 pad 3: /MOSI -> /MISO
- U5 pad 4: /MOSI_1.8V -> /MISO_1.8V
- U5 pad 6: /MISO -> /CSB
Routing:
- net +3.3V: track 9.71 -> 31.7 mm, vias 3 -> 4
- net /CS_1.8V: track 9.38 -> 16.6 mm
- net /MISO: track 5.27 -> 10.4 mm, vias 0 -> 1
- net /SCLK: track 6.07 -> 10.6 mm
- net GND: track 12.2 -> 16.6 mm, vias 0 -> 12
- net /MOSI: track 8.17 -> 5.37 mm
- net /MOSI_1.8V: track 7.30 -> 9.25 mm
- net /SCK_1.8V: track 8.10 -> 9.90 mm
- net /CSB: track 10.0 -> 9.01 mm
- net Net-(U4-REGOUT): track 1.23 -> 2.03 mm
- net /1.8V: track 27.2 -> 27.6 mm, vias 4 -> 2
- added copper zone on B.Cu, net GND
- removed copper zone on B.Cu, net +3.3V

Commit message: updated
Parts:
- added REF**: logo_aightech, 00_custom-footprints:logo_aightech, B.Cu at (26.1, 35.0)
- added kibuzzard-66093797: G***, kibuzzard-66093797, B.Cu at (33.1, 32.5)
Other:
- board text added: "ClvHd IMU"

Commit message: renamed SPI buses
Connections:
- net /MISO renamed /POCI
- net /MISO_1.8V renamed /POCI_1.8V
- net /MOSI renamed /PICO
- net /MOSI_1.8V renamed /PICO_1.8V
- net /MOSI_ARM renamed /PICO_ARM
- net /SWDIO/MISO_ARM renamed /SWDIO/POCI_ARM
Changed lines of the file:
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@@
 	(net 3 "/extRef")
 	(net 4 "unconnected-(J3-Pin_1-Pad1)")
-	(net 5 "/MISO")
-	(net 6 "/MOSI")
+	(net 5 "/POCI")
+	(net 6 "/PICO")
 	(net 7 "/SCLK")
 	(net 8 "/CSB")
 	(net 9 "/1.8V")
 	(net 10 "/SCK_1.8V")
-	(net 11 "/MOSI_1.8V")
-	(net 12 "/MISO_1.8V")
+	(net 11 "/PICO_1.8V")
+	(net 12 "/POCI_1.8V")
 	(net 13 "unconnected-(U4-NC-Pad4)")
 	(net 14 "unconnected-(U4-INT1-Pad12)")
@@
 	(net 28 "unconnected-(U4-AUX_DA-Pad21)")
 	(net 29 "/IO1_out")
-	(net 30 "/SWDIO{slash}MISO_ARM")
-	(net 31 "/MOSI_ARM")
+	(net 30 "/SWDIO{slash}POCI_ARM")
+	(net 31 "/PICO_ARM")
 	(net 32 "/SCLK_ARM")
 	(net 33 "/SPICS_ARM")
@@
 			(layers "F.Cu" "F.Paste" "F.Mask")
 			(roundrect_rratio 0.25)
-			(net 5 "/MISO")
+			(net 5 "/POCI")
 			(pintype "passive")
 		)
@@
 			(layers "F.Cu" "F.Paste" "F.Mask")
 			(roundrect_rratio 0.25)
-			(net 6 "/MOSI")
+			(net 6 "/PICO")
 			(pintype "passive")
 		)
@@
 			(layers "*.Cu" "*.Mask")
 			(remove_unused_layers no)
-			(net 6 "/MOSI")
+			(net 6 "/PICO")
 			(pinfunction "Pin_1")
 			(pintype "passive")
@@
 			(size 0.35 0.92)
 			(layers "F.Cu" "F.Paste" "F.Mask")
-			(net 5 "/MISO")
+			(net 5 "/POCI")
 			(pinfunction "D1")
 			(pintype "output")
@@
 			(size 0.35 0.92)
 			(layers "F.Cu" "F.Paste" "F.Mask")
-			(net 12 "/MISO_1.8V")
+			(net 12 "/POCI_1.8V")
 			(pinfunction "S1")
 			(pintype "input")
@@
 			(layers "*.Cu" "*.Mask")
 			(remove_unused_layers no)
-			(net 30 "/SWDIO{slash}MISO_ARM")
+			(net 30 "/SWDIO{slash}POCI_ARM")
 			(pinfunction "Pin_1")
 			(pintype "passive")
@@
 			(layers "F.Cu" "F.Paste" "F.Mask")
 			(roundrect_rratio 0.25)
-			(net 12 "/MISO_1.8V")
+			(net 12 "/POCI_1.8V")
 			(pinfunction "SDO/AD0")
 			(pintype "unspecified")
@@
 			(size 0.115147 0.115147)
 			(layers "F.Cu" "F.Paste" "F.Mask")
-			(net 11 "/MOSI_1.8V")
+			(net 11 "/PICO_1.8V")
 			(pinfunction "SDA/SDI")
 			(pintype "unspecified")
@@
 			(layers "F.Cu" "F.Paste" "F.Mask")
 			(roundrect_rratio 0.25)
-			(net 12 "/MISO_1.8V")
+			(net 12 "/POCI_1.8V")
 			(pintype "passive")
 		)
@@
 			(layers "*.Cu" "*.Mask")
 			(remove_unused_layers no)
-			(net 5 "/MISO")
+			(net 5 "/POCI")
 			(pinfunction "Pin_1")
 			(pintype "passive")
@@
 			(layers "F.Cu" "F.Paste" "F.Mask")
 			(roundrect_rratio 0.25)
-			(net 11 "/MOSI_1.8V")
+			(net 11 "/PICO_1.8V")
 			(pintype "passive")
 		)
@@
 			(size 0.35 0.92)
 			(layers "F.Cu" "F.Paste" "F.Mask")
-			(net 6 "/MOSI")
+			(net 6 "/PICO")
 			(pinfunction "D1")
 			(pintype "output")
@@
 			(size 0.35 0.92)
 			(layers "F.Cu" "F.Paste" "F.Mask")
-			(net 11 "/MOSI_1.8V")
+			(net 11 "/PICO_1.8V")
 			(pinfunction "S1")
 			(pintype "input")
@@
 			(layers "*.Cu" "*.Mask")
 			(remove_unused_layers no)
-			(net 31 "/MOSI_ARM")
+			(net 31 "/PICO_ARM")
 			(pinfunction "Pin_1")
 			(pintype "passive")
