File: KiCad/modules/VIB_STSPIN240/VIB_STSPIN240.kicad_sch (KiCad schematic)
At the start: 39 parts, among them J10 Conn_01x01_Pin, J11 Conn_01x01_Pin, J12 Conn_01x01_Pin, J13 Conn_01x01_Pin, J14 Conn_01x01_Pin, J15 Conn_01x01_Pin, J16 Conn_01x01_Pin, J17 Conn_01x01_Pin, J18 Conn_01x01_Pin, J19 Conn_01x01_Pin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

Commit message: renamed SPI buses
Connections:
- net MISO renamed POCI
- net MOSI renamed PICO
- net MOSI_ARM renamed PICO_ARM
Changed lines of the file:
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@@
 		)
 	)
-	(label "MOSI_ARM"
+	(label "PICO_ARM"
 		(at 254 106.68 180)
 		(fields_autoplaced yes)
@@
 		)
 	)
-	(label "MOSI"
+	(label "PICO"
 		(at 88.9 55.88 270)
 		(fields_autoplaced yes)
@@
 		)
 	)
-	(label "MISO"
+	(label "POCI"
 		(at 86.36 55.88 270)
 		(fields_autoplaced yes)
