File: KiCad/modules/DRY_FLEX/DRY_FLEX.kicad_pcb (KiCad board)
At the start: 2 copper layers, 91 x 100 mm, 67 parts, among them J1 Conn_01x01_Pin, J10 Conn_01x01_Pin, J11 Conn_01x01_Pin, J12 Conn_01x01_Pin, J13 Conn_01x01_Pin, J14 Conn_01x01_Pin, J15 Conn_01x01_Pin, J16 Conn_01x01_Pin, J17 Conn_01x01_Pin, J18 Conn_01x01_Pin, J19 Conn_01x01_Pin, J2 Conn_01x01_Pin, J20 Conn_01x01_Pin, J21 Conn_01x01_Pin, J22 Conn_01x01_Pin, J23 Conn_01x01_Pin, J24 Conn_01x01_Pin, J25 Conn_01x01_Pin, J26 Conn_01x01_Pin, J27 Conn_01x01_Pin, J28 Conn_01x01_Pin, J29 Conn_01x01_Pin, J3 Conn_01x01_Pin, J30 Conn_01x01_Pin, J31 Conn_01x01_Pin, J32 Conn_01x01_Pin, J4 Conn_01x01_Pin, J5 Conn_01x01_Pin, J6 Conn_01x01_Pin, J7 Conn_01x01_Pin, J8 Conn_01x01_Pin, J9 Conn_01x01_Pin

Commit message: update
Routing:
- net /in1-: track 76.3 -> 103.5 mm
- net /in2-: track 62.9 -> 90.0 mm
- net /in3-: track 56.8 -> 84.0 mm
- net /in4-: track 51.6 -> 78.7 mm
- net /in5-: track 51.7 -> 78.7 mm
- net /in6-: track 56.3 -> 83.3 mm
- net /in7-: track 63.2 -> 90.2 mm
- net /in1+: track 76.2 -> 103.2 mm
- net /in6+: track 59.4 -> 86.4 mm
- net /in3+: track 59.8 -> 86.8 mm
- net /in7+: track 63.6 -> 90.6 mm
- net /in5+: track 44.5 -> 71.5 mm
- net /in2+: track 63.1 -> 90.1 mm
- net /in4+: track 44.5 -> 71.5 mm
