File: KiCad/modules/DRY_ELEC_6CH_THIN/DRY_ELEC_6CH_THIN.kicad_pcb (KiCad board)
At the start: 4 copper layers, 30 x 9 mm, 53 parts, among them J1 Conn_01x01_Pin, J10 Conn_01x01_Pin, J11 Conn_01x01_Pin, J12 Conn_01x01_Pin, J13 Conn_01x01_Pin, J14 Conn_01x01_Pin, J15 Conn_01x01_Pin, J16 Conn_01x01_Pin, J17 Conn_01x01_Pin, J18 Conn_01x01_Pin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

Commit message: added mid size to fit better with ads1293 module and standad xtal + some modificaion
Parts:
- moved kibuzzard-66BB0EE4 14.2 mm to (15.8, 32.1), turned to 90 degrees
- moved J16 0.07 mm to (34.4, 28.7)
- moved J9 0.07 mm to (25.6, 28.7)
- moved J1 0.06 mm to (25.6, 27.3)
- moved J8 0.06 mm to (34.4, 27.3)
