File: KiCad/controller/CONTROLLER_XIAO/CONTROLLER_XIAO.kicad_pcb (KiCad board)
At the start: 4 copper layers, 20 x 20.5 mm, 8 parts, among them J1 Conn_01x02_Pin, J3 Conn_01x02_Pin, U2 SEEEDUINO-XIAO-ESP32C3

Commit message: updated
Parts:
- added U1: MCP4728A0T-E/UNVAO, 00_lcsc:MSOP-10_L3.0-W3.0-P0.50-LS5.0-BL, B.Cu at (51.3, 80.9)
- moved U2 9.00 mm to (56.5, 94.7)
Other:
- outline, holes or cut-outs redrawn
