File: pcb/hmi/submodule/sensor/EMG_INA331/EMG_INA331.kicad_pcb (KiCad board)
At the start: 4 copper layers, 15 x 11 mm, 50 parts, among them J1 Conn_01x01_Pin, J10 Conn_01x01_Pin, J11 Conn_01x01_Pin, J12 Conn_01x01_Pin, J2 Conn_01x01_Pin, J3 Conn_01x01_Pin, J4 Conn_01x01_Pin, J5 Conn_01x01_Pin, J6 Conn_01x01_Pin, J7 Conn_01x01_Pin, J8 Conn_01x01_Pin, J9 Conn_01x01_Pin, U1 INA331IDGKR, U2 OPA333, U3 AP2112K-3.3TRG1, U4 OPA333, U5 CJ432, U6 LIS3DHTR

Commit message: feat(EMG_INA331): drop the LIS3DH, keep the module INA331-only
The accelerometer moves out to the new EMG_INA331_LIS variant so that
EMG_INA331 is a plain analog EMG front-end usable with any ADC-capable
com module. All 7 LIS3DH references are gone from the schematic.

Also fixes the outstanding ERC issues: U6 pin 13 (ADC3) is no longer
dangling and the power symbols are re-synced with the library, taking
the report from 6 errors / 55 warnings down to 5 / 23. DRC stays at 0
violations. Plots, PDF, SVG and DRC/ERC logs regenerated under KiCad 10.

Claude-Session: https://claude.ai/code/session_01Fp1CWL3JE8kAHQpHzFCsU5
Parts:
- removed C14: 100nF, Capacitor_SMD:C_0402_1005Metric
- removed C15: 1uF, Capacitor_SMD:C_0402_1005Metric
- removed TP1, TP2: TestPoint, 00_custom-footprints:TestPoint_Pad_D1.0mm
- removed U6: LIS3DHTR, 00_lcsc:LGA-16_L3.0-W3.0-P0.50-TL
- added J13: Conn_01x01_Pin, 00_custom-footprints:PinHeader_1x01_P1.27mm_Vertical, F.Cu at (35.7, 27.0)
- moved R14 3.29 mm to (34.0, 29.4), turned to 180 degrees
Routing:
- net +3.3V: track 32.3 -> 10.2 mm, vias 1 -> 0
- net +3.3VA: track 39.6 -> 28.8 mm, vias 2 -> 3
- net GND: track 24.7 -> 15.9 mm, vias 9 -> 8
- net /SCLK: track 7.14 -> 0.00 mm
- net /POCI: track 6.35 -> 0.00 mm
- net /PICO: track 5.52 -> 0.00 mm
- net /ADC2: track 5.49 -> 0.00 mm, vias 1 -> 0
- net Vref: track 29.0 -> 24.5 mm, vias 2 -> 1
- net /CSB: track 2.63 -> 0.00 mm, vias 1 -> 0
- net /OUT1: track 10.1 -> 11.6 mm
- net /extRef: track 1.24 -> 2.50 mm
