File: pcb/hmi/submodule/sensor/EMG_INA331/EMG_INA331.kicad_sch (KiCad schematic)
At the start: 49 parts, among them J1 Conn_01x01_Pin, J10 Conn_01x01_Pin, J11 Conn_01x01_Pin, J12 Conn_01x01_Pin, J2 Conn_01x01_Pin, J3 Conn_01x01_Pin, J4 Conn_01x01_Pin, J5 Conn_01x01_Pin, J6 Conn_01x01_Pin, J7 Conn_01x01_Pin, J8 Conn_01x01_Pin, J9 Conn_01x01_Pin, U1 INA331IDGKR, U2 OPA333, U3 AP2112K-3.3TRG1, U4 OPA333, U5 CJ432, U6 LIS3DHTR

Commit message: feat(EMG_INA331): drop the LIS3DH, keep the module INA331-only
The accelerometer moves out to the new EMG_INA331_LIS variant so that
EMG_INA331 is a plain analog EMG front-end usable with any ADC-capable
com module. All 7 LIS3DH references are gone from the schematic.

Also fixes the outstanding ERC issues: U6 pin 13 (ADC3) is no longer
dangling and the power symbols are re-synced with the library, taking
the report from 6 errors / 55 warnings down to 5 / 23. DRC stays at 0
violations. Plots, PDF, SVG and DRC/ERC logs regenerated under KiCad 10.

Claude-Session: https://claude.ai/code/session_01Fp1CWL3JE8kAHQpHzFCsU5
Parts:
- removed C14: 100nF, Capacitor_SMD:C_0402_1005Metric, symbol Device:C
- removed C15: 1uF, Capacitor_SMD:C_0402_1005Metric, symbol Device:C
- removed TP1, TP2: TestPoint, 00_custom-footprints:TestPoint_Pad_D1.0mm, symbol 00_custom:TestPoint
- removed U6: LIS3DHTR, 00_lcsc:LGA-16_L3.0-W3.0-P0.50-TL, symbol 00_lcsc:LIS3DHTR
- added J13: Conn_01x01_Pin, 00_custom-footprints:PinHeader_1x01_P1.27mm_Vertical, symbol Connector:Conn_01x01_Pin
Connections:
- net OUT1: now also J13.1 (Pin_1)
- no-connect marks 5 -> 1
